File: EncoderBoard/EncoderBoard.sch (KiCad schematic (older format))
At the start: 39 parts

Commit message: Updated all switches to LED. Added EEPROM. Added rough costing.
Decided all switches could be LED (I can work out the colours later).
The EEPROM is a 1Mb model - might come in handy later.
Rough Costs was just to get a decent sense of how much this project will actually cost. Thankfully I already have some Pis...
Parts:
- added U?: CAT24M01W, Package_SO:SOIC-8_3.9x4.9mm_P1.27mm, symbol Memory_EEPROM:CAT24M01W
Connections:
- net +3V3: now also U?.8 (VCC)
- net +5V: now also U?.1 (A->B)
- net GND: now also U?.10 (GND), U?.19 (CE), U?.2 (A1), U?.3 (A2), U?.4 (GND)
- net INT0_A: now also U?.20 (INTA); no longer U?.19 (INTB)
- net INT0_B: now also U?.19 (INTB); no longer U?.20 (INTA)
- net INT1_A: now also U?.20 (INTA); no longer U?.19 (INTB)
- net INT1_B: now also U?.19 (INTB); no longer U?.20 (INTA)
- net INT2_A: now also U?.20 (INTA); no longer U?.19 (INTB)
- net INT2_B: now also U?.19 (INTB); no longer U?.20 (INTA)
- net SCL: now also U?.6 (SCL)
- net SDA: now also U?.5 (SDA)
- net WS2812_DATA: now reaches R?.1
- new net EEPROM_WP: U?.7 (WP)
- no-connect marks 24 -> 52
Other:
- moved on the sheet: C?, R?, U?
Changed lines of the file:
@@
 ENC8_SW
 $Sheet
-S 5300 6050 500  150
+S 10050 5700 500  150
 U 5CFF3BEB
 F0 "Encoders and Buttons" 50
@@
 Text GLabel 5850 1300 0    50   Input ~ 0
 CS2
+Text GLabel 850  2000 0    50   Input ~ 0
+INT0_A
 Text GLabel 850  1900 0    50   Input ~ 0
-INT0_A
-Text GLabel 850  2000 0    50   Input ~ 0
 INT0_B
+Text GLabel 3350 2000 0    50   Input ~ 0
+INT1_A
 Text GLabel 3350 1900 0    50   Input ~ 0
-INT1_A
-Text GLabel 3350 2000 0    50   Input ~ 0
 INT1_B
+Text GLabel 5850 2000 0    50   Input ~ 0
+INT2_A
 Text GLabel 5850 1900 0    50   Input ~ 0
-INT2_A
-Text GLabel 5850 2000 0    50   Input ~ 0
 INT2_B
 Wire Wire Line
@@
 Wire Wire Line
 	3250 2200 3250 2700
-Connection ~ 3250 2700
 Wire Wire Line
 	5850 2200 5750 2200
@@
 Connection ~ 6550 750
 $Sheet
-S 5300 6600 500  150
+S 10050 6250 500  150
 U 5D4582C3
 F0 "Displays and LEDs" 50
@@
 L 74xx:74HC245 U?
 U 1 1 5D4D59BC
-P 5350 4800
-F 0 "U?" H 5350 5781 50  0000 C CNN
-F 1 "74HCT245" H 5350 5690 50  0000 C CNN
-F 2 "" H 5350 4800 50  0001 C CNN
-F 3 "http://www.ti.com/lit/gpn/sn74HC245" H 5350 4800 50  0001 C CNN
-	1    5350 4800
+P 5100 4500
+F 0 "U?" H 5100 5481 50  0000 C CNN
+F 1 "74HCT245" H 5100 5390 50  0000 C CNN
+F 2 "" H 5100 4500 50  0001 C CNN
+F 3 "http://www.ti.com/lit/gpn/sn74HC245" H 5100 4500 50  0001 C CNN
+	1    5100 4500
 	1    0    0    -1
 $EndComp
@@
 L Device:R R?
 U 1 1 5D4D6EBC
-P 6100 4300
-F 0 "R?" V 5893 4300 50  0000 C CNN
-F 1 "330R" V 5984 4300 50  0000 C CNN
-F 2 "" V 6030 4300 50  0001 C CNN
-F 3 "~" H 6100 4300 50  0001 C CNN
-	1    6100 4300
+P 5850 4000
+F 0 "R?" V 5643 4000 50  0000 C CNN
+F 1 "330R" V 5734 4000 50  0000 C CNN
+F 2 "" V 5780 4000 50  0001 C CNN
+F 3 "~" H 5850 4000 50  0001 C CNN
+	1    5850 4000
 	0    1    1    0
 $EndComp
 Wire Wire Line
-	5950 4300 5850 4300
-Text Label 4850 4300 2    50   ~ 0
+	5700 4000 5600 4000
+Text Label 4600 4000 2    50   ~ 0
 WS2812_3V3
 Text Label 1700 6800 2    50   ~ 0
@@
 L power:+5V #PWR0146
 U 1 1 5D4E0E6E
-P 5350 3750
-F 0 "#PWR0146" H 5350 3600 50  0001 C CNN
-F 1 "+5V" H 5365 3923 50  0000 C CNN
-F 2 "" H 5350 3750 50  0001 C CNN
-F 3 "" H 5350 3750 50  0001 C CNN
-	1    5350 3750
+P 5100 3450
+F 0 "#PWR0146" H 5100 3300 50  0001 C CNN
+F 1 "+5V" H 5115 3623 50  0000 C CNN
+F 2 "" H 5100 3450 50  0001 C CNN
+F 3 "" H 5100 3450 50  0001 C CNN
+	1    5100 3450
 	1    0    0    -1
 $EndComp
@@
 L Device:C_Small C?
 U 1 1 5D4E181A
-P 5700 3850
-F 0 "C?" H 5792 3896 50  0000 L CNN
-F 1 "100nF" H 5792 3805 50  0000 L CNN
-F 2 "" H 5700 3850 50  0001 C CNN
-F 3 "~" H 5700 3850 50  0001 C CNN
-	1    5700 3850
-	1    0    0    -1
-$EndComp
-Wire Wire Line
-	5700 3750 5350 3750
-Wire Wire Line
-	5350 4000 5350 3750
-Connection ~ 5350 3750
+P 5450 3550
+F 0 "C?" H 5542 3596 50  0000 L CNN
+F 1 "100nF" H 5542 3505 50  0000 L CNN
+F 2 "" H 5450 3550 50  0001 C CNN
+F 3 "~" H 5450 3550 50  0001 C CNN
+	1    5450 3550
+	1    0    0    -1
+$EndComp
+Wire Wire Line
+	5450 3450 5100 3450
+Wire Wire Line
+	5100 3700 5100 3450
+Connection ~ 5100 3450
 $Comp
 L power:GND #PWR0147
 U 1 1 5D4F02EF
-P 5700 3950
-F 0 "#PWR0147" H 5700 3700 50  0001 C CNN
-F 1 "GND" H 5705 3777 50  0000 C CNN
-F 2 "" H 5700 3950 50  0001 C CNN
-F 3 "" H 5700 3950 50  0001 C CNN
-	1    5700 3950
+P 5450 3650
+F 0 "#PWR0147" H 5450 3400 50  0001 C CNN
+F 1 "GND" H 5455 3477 50  0000 C CNN
+F 2 "" H 5450 3650 50  0001 C CNN
+F 3 "" H 5450 3650 50  0001 C CNN
+	1    5450 3650
 	1    0    0    -1
 $EndComp
@@
 	3850 7100 3700 7100
 NoConn ~ 3700 6900
+Connection ~ 3250 2700
+Text GLabel 6000 4000 2    50   Input ~ 0
+WS2812_DATA
+NoConn ~ 9350 4700
+NoConn ~ 9350 4800
+NoConn ~ 9350 4900
+NoConn ~ 9350 5000
+NoConn ~ 9350 5100
+NoConn ~ 9350 5200
+NoConn ~ 9350 5300
+NoConn ~ 9350 5400
+NoConn ~ 9350 5500
+NoConn ~ 9350 5600
+NoConn ~ 9350 5700
+NoConn ~ 9350 5800
+NoConn ~ 9350 5900
+NoConn ~ 9350 6000
+NoConn ~ 5600 4700
+NoConn ~ 5600 4600
+NoConn ~ 5600 4500
+NoConn ~ 5600 4400
+NoConn ~ 5600 4300
+NoConn ~ 5600 4200
+NoConn ~ 5600 4100
+NoConn ~ 4600 4700
+NoConn ~ 4600 4600
+NoConn ~ 4600 4500
+NoConn ~ 4600 4400
+NoConn ~ 4600 4300
+NoConn ~ 4600 4200
+NoConn ~ 4600 4100
+$Comp
+L power:GND #PWR?
+U 1 1 5D090AE0
+P 5100 5300
+F 0 "#PWR?" H 5100 5050 50  0001 C CNN
+F 1 "GND" H 5105 5127 50  0000 C CNN
+F 2 "" H 5100 5300 50  0001 C CNN
+F 3 "" H 5100 5300 50  0001 C CNN
+	1    5100 5300
+	1    0    0    -1
+$EndComp
+$Comp
+L power:+5V #PWR?
+U 1 1 5D091459
+P 4450 4900
+F 0 "#PWR?" H 4450 4750 50  0001 C CNN
+F 1 "+5V" H 4465 5073 50  0000 C CNN
+F 2 "" H 4450 4900 50  0001 C CNN
+F 3 "" H 4450 4900 50  0001 C CNN
+	1    4450 4900
+	1    0    0    -1
+$EndComp
+$Comp
+L power:GND #PWR?
+U 1 1 5D0920A0
+P 4450 5000
+F 0 "#PWR?" H 4450 4750 50  0001 C CNN
+F 1 "GND" H 4455 4827 50  0000 C CNN
+F 2 "" H 4450 5000 50  0001 C CNN
+F 3 "" H 4450 5000 50  0001 C CNN
+	1    4450 5000
+	1    0    0    -1
+$EndComp
+Wire Wire Line
+	4450 5000 4600 5000
+Wire Wire Line
+	4600 4900 4450 4900
+$Comp
+L Memory_EEPROM:CAT24M01W U?
+U 1 1 5CF5D347
+P 5600 6250
+F 0 "U?" H 5600 6731 50  0000 C CNN
+F 1 "CAT24M01W" H 5600 6640 50  0000 C CNN
+F 2 "Package_SO:SOIC-8_3.9x4.9mm_P1.27mm" H 6450 6000 50  0001 C CNN
+F 3 "https://www.onsemi.com/pub/Collateral/CAT24M01-D.PDF" H 5600 6250 50  0001 C CNN
+	1    5600 6250
+	1    0    0    -1
+$EndComp
+Text GLabel 6000 6150 2    50   Input ~ 0
+SDA
+Text GLabel 6000 6250 2    50   Input ~ 0
+SCL
+Text GLabel 6000 6350 2    50   Input ~ 0
+EEPROM_WP
+$Comp
+L power:GND #PWR?
+U 1 1 5CF60E9A
+P 5100 6400
+F 0 "#PWR?" H 5100 6150 50  0001 C CNN
+F 1 "GND" H 5105 6227 50  0000 C CNN
+F 2 "" H 5100 6400 50  0001 C CNN
+F 3 "" H 5100 6400 50  0001 C CNN
+	1    5100 6400
+	1    0    0    -1
+$EndComp
+Wire Wire Line
+	5200 6350 5100 6350
+Wire Wire Line
+	5100 6350 5100 6400
+Wire Wire Line
+	5200 6250 5100 6250
+Wire Wire Line
+	5100 6250 5100 6350
+Connection ~ 5100 6350
+$Comp
+L power:GND #PWR?
+U 1 1 5CF71724
+P 5600 6550
+F 0 "#PWR?" H 5600 6300 50  0001 C CNN
+F 1 "GND" H 5605 6377 50  0000 C CNN
+F 2 "" H 5600 6550 50  0001 C CNN
+F 3 "" H 5600 6550 50  0001 C CNN
+	1    5600 6550
+	1    0    0    -1
+$EndComp
+$Comp
+L power:+3V3 #PWR?
+U 1 1 5CF71FF6
+P 5600 5700
+F 0 "#PWR?" H 5600 5550 50  0001 C CNN
+F 1 "+3V3" H 5615 5873 50  0000 C CNN
+F 2 "" H 5600 5700 50  0001 C CNN
+F 3 "" H 5600 5700 50  0001 C CNN
+	1    5600 5700
+	1    0    0    -1
+$EndComp
+Wire Wire Line
+	5600 5700 5600 5950
 $EndSCHEMATC

Commit message: Generated draft footprint PCB with (very) approximate placements.
Parts:
- C1, C10, C3, C5, C7, C9: renamed from C?; footprint (none) -> Capacitor_BG:C_0805_2012Metric
- C11, C2, C4, C6, C8: renamed from C?; footprint (none) -> Capacitor_BG:C_1210_3225Metric
- R1, R10, R11, R12, R13, R14, R15, R16, R17, R18, R19, R2, R20, R21, R3, R4, R5, R6, R7, R8, R9: renamed from R?; footprint (none) -> Resistor_BG:R_0805_2012Metric
- U1, U2, U3: renamed from U?; footprint Package_SO:SOIC-28W_7.5x17.9mm_P1.27mm -> SOIC_BG:SOIC-28W_7.5x17.9mm_P1.27mm; symbol Interface_Expansion:MCP23S17_SO -> Interface_Expansion_BG:MCP23S17_SO
- U4, U6: renamed from U?; footprint Package_SO:TSSOP-24_4.4x7.8mm_P0.65mm -> TSSOP_BG:TSSOP-24_4.4x7.8mm_P0.65mm
- U5: renamed from U?; footprint (none) -> SOIC_BG:SOIC-20W_7.5x12.8mm_P1.27mm
- U7: renamed from U?; footprint (none) -> Teensy_BG:Teensy30_31_32_LC; symbol Teensy:Teensy3.2 -> Teensy_BG:Teensy3.2
- U8: renamed from U?; footprint Package_SO:SOIC-8_3.9x4.9mm_P1.27mm -> SOIC_BG:SOIC-8_3.9x4.9mm_P1.27mm
Connections:
- net RST2 is gone; now on net EEPROM_WP: U7.4 (2)
- net RST3 is gone; now on net INT0_A: U7.5 (3_TX_PWM)
- net RST4 is gone; now on net INT0_B: U7.6 (4_RX_PWM)
- net RST7 is gone; now on net INT1_A: U7.9 (7_RX3_DOUT)
- net RST8 is gone; now on net INT1_B: U7.10 (8_TX3_DIN)
- net INT2_A: now also U7.23 (16_A2_SCL0_Touch)
- net INT2_B: now also U7.24 (17_A3_SDA0_Touch)
- net RST0: no longer names the net of U7.2 (0_RX1_Touch)
- net RST1: no longer names the net of U7.3 (1_TX1_Touch)
- net RST5 renamed BUTTON0_LED
- net RST6 renamed BUTTON1_LED
- no-connect marks 52 -> 72

Commit message: Tidied up the encoder board, updated debounce logic for schematic.
Parts:
- added U? (x3): CAT24M01W, SOIC_BG:SOIC-8_3.9x4.9mm_P1.27mm, symbol Memory_EEPROM:CAT24M01W
Connections:
- net +3V3: now also U1.18 (~RESET~), U2.18 (~RESET~), U3.18 (~RESET~), U6.1 (A0), U?.2 (A1), U?.2 (A1), U?.3 (A2), U?.3 (A2), U?.8 (VCC), U?.8 (VCC), U?.8 (VCC)
- net EEPROM_WP: now also U?.7 (WP), U?.7 (WP), U?.7 (WP)
- net GND: now also U?.2 (A1), U?.3 (A2), U?.4 (GND), U?.4 (GND), U?.4 (GND); no longer U1.18 (~RESET~), U2.18 (~RESET~), U3.18 (~RESET~), U6.1 (A0)
- net INT0_A: now also U7.9 (7_RX3_DOUT); no longer U7.5 (3_TX_PWM)
- net INT1_A: now also U7.10 (8_TX3_DIN); no longer U7.9 (7_RX3_DOUT)
- net INT2_A: now also U7.11 (9_RX2_CS_PWM); no longer U7.23 (16_A2_SCL0_Touch)
- net SCL: now also U?.6 (SCL), U?.6 (SCL), U?.6 (SCL)
- net SDA: now also U?.5 (SDA), U?.5 (SDA), U?.5 (SDA)
- net WS2812_3V3: now also U7.3 (1_TX1_Touch); no longer U7.21 (14_A0_SCK)
- net CS1: no longer names the net of U2.11 (~CS~)
- net CS1: no longer U7.11 (9_RX2_CS_PWM)
- net CS2: no longer names the net of U7.22 (15_A1_CS_Touch)
- net CS2: no longer U3.11 (~CS~)
- net INT0_B: no longer names the net of U7.6 (4_RX_PWM)
- net INT0_B: no longer U1.19 (INTB)
- net INT1_B: no longer names the net of U2.19 (INTB)
- net INT1_B: no longer U7.10 (8_TX3_DIN)
- net INT2_B: no longer names the net of U7.24 (17_A3_SDA0_Touch)
- net INT2_B: no longer U3.19 (INTB)
- no-connect marks 72 -> 79
Other:
- moved on the sheet: U8
