File: EncoderBoard/Displays&LEDs.sch (KiCad schematic (older format))
At the start: 33 parts

Commit message: Updated schematic with appropriate symbols and latest library.
Connections:
- net labels removed: RST0, RST1, RST2, RST3, RST4, RST5, RST6, RST7, RST8
- wire segments 45 -> 36
- no-connect marks 10 -> 1
Other:
- moved on the sheet: C?, D?, U?

Commit message: Generated draft footprint PCB with (very) approximate placements.
Parts:
- C30, C31, C32, C33, C34, C35, C36, C37, C38, C39, C40, C41: renamed from C?; footprint (none) -> Capacitor_BG:C_0805_2012Metric
- D1, D10, D11, D12, D2, D3, D4, D5, D6, D7, D8, D9: renamed from D?; footprint LED_SMD:LED_WS2812B_PLCC4_5.0x5.0mm_P3.2mm -> LED_BG:LED_WS2812B_PLCC4_5.0x5.0mm_P3.2mm
- U10, U11, U12, U13, U14, U15, U16, U17, U9: renamed from U?; footprint MODULE -> Display_BG:Display_OLED_128x32_I2C; symbol Displays:Display_OLED_128x32_I2C -> Displays_BG:Display_OLED_128x32_I2C

Commit message: Final version of Rev A board.
- Fixed up address pins on some chips.
- Added some additional bypass capacitors.
- Fixed up some broken footprint references.
- Some minor layout adjustments.
Parts:
- added C63, C64, C65, C66, C67, C68, C69, C70, C71: 100nF, Capacitor_BG:C_0805_2012Metric, symbol Device:C_Small
Connections:
- net +3V3: now also C63.1, C64.1, C65.1, C66.1, C67.1, C68.1, C69.1, C70.1, C71.1
- net GND: now also C63.2, C64.2, C65.2, C66.2, C67.2, C68.2, C69.2, C70.2, C71.2
