File: EncoderBoard/EncoderBoard.kicad_pcb (KiCad board)
At the start: 2 copper layers, 221 x 61 mm, 216 parts, among them SW1 Rotary_Encoder_Switch, SW10 SW_Push_LED_Red, SW11 SW_Push_LED_Blue, SW12 SW_Push_LED_Red, SW13 SW_Push_LED_Yellow, SW14 SW_Push_LED_Green, SW15 SW_Push_LED_Blue, SW2 Rotary_Encoder_Switch, SW3 Rotary_Encoder_Switch, SW4 Rotary_Encoder_Switch, SW5 Rotary_Encoder_Switch, SW6 Rotary_Encoder_Switch, SW7 Rotary_Encoder_Switch, SW8 Rotary_Encoder_Switch, SW9 Rotary_Encoder_Switch, U1 MCP23S17_SO, U10 Display_OLED_128x32_I2C, U11 Display_OLED_128x32_I2C, U12 Display_OLED_128x32_I2C, U13 Display_OLED_128x32_I2C, U14 Display_OLED_128x32_I2C, U15 Display_OLED_128x32_I2C, U16 Display_OLED_128x32_I2C, U17 Display_OLED_128x32_I2C, U18 74LVC14, U19 74LCV14, U2 MCP23S17_SO, U20 74LVC14, U21 74LVC14, U22 74LVC14, U23 74LVC14, U24 CAT24M01W, U25 CAT24M01W, U26 CAT24M01W, U3 MCP23S17_SO, U4 TCA9548APWR, U5 74HCT245, U6 TCA9548APWR, U7 Teensy3.2, U8 CAT24M01W, U9 Display_OLED_128x32_I2C

Commit message: Final version of Rev A board.
- Fixed up address pins on some chips.
- Added some additional bypass capacitors.
- Fixed up some broken footprint references.
- Some minor layout adjustments.
Parts:
- added C72: 100nF, Capacitor_BG:C_0805_2012Metric, B.Cu at (208.8, 55.1)
- added C73: 100nF, Capacitor_BG:C_0805_2012Metric, B.Cu at (219.7, 65.5)
- added C74: 100nF, Capacitor_BG:C_0805_2012Metric, B.Cu at (210.2, 68.2)
- added C75: 100nF, Capacitor_BG:C_0805_2012Metric, B.Cu at (219.8, 78.0)
- added R88: 4.7k, Resistor_BG:R_0805_2012Metric, F.Cu at (133.6, 84.5)
- added R89: 4.7k, Resistor_BG:R_0805_2012Metric, F.Cu at (211.5, 83.1)
- C12, C13, C16, C17, C21, C22, C23, C24, C29, C42, C43, C44, C48, C49, C50, C51, C55, C56: value 0.01uF -> 10nF
- C14, C15, C18, C19, C20, C25, C26, C27, C28, C45, C46, C47, C52, C53, C54, C57, C58, C59, C60, C61, C62: value 0.1uF -> 100nF
- moved C6 70.7 mm to (266.5, 88.1)
- moved U2 70.7 mm to (171.6, 74.5)
- moved U4 70.7 mm to (137.1, 91.0)
- moved C1 70.7 mm to (100.5, 77.0)
- moved C10 70.7 mm to (214.9, 85.8)
- moved C11 70.7 mm to (214.9, 83.0)
- moved C12 70.7 mm to (72.5, 64.5)
- moved C13 70.7 mm to (75.0, 64.5)
- moved C14 70.7 mm to (71.0, 56.5)
- moved C15 70.7 mm to (110.0, 84.5)
- moved C16 70.7 mm to (111.5, 92.5)
- moved C17 70.7 mm to (113.5, 92.5)
- moved C18 70.7 mm to (263.2, 85.0)
- moved C19 70.7 mm to (110.0, 56.5)
- moved C2 70.7 mm to (103.1, 77.0)
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Connections:
- U2 pad 15: GND -> +3V3
- U3 pad 16: GND -> +3V3
- U4 pad 3: GND -> Net-(R88-Pad2)
- U6 pad 3: GND -> Net-(R89-Pad2)
Routing:
- net +3V3: track 984.3 -> 1021.8 mm
- net Net-(R89-Pad2): track 0.00 -> 6.63 mm
- net GND: track 706.4 -> 711.1 mm, vias 36 -> 38
- net SCL: track 191.5 -> 196.0 mm
- net Net-(R88-Pad2): track 0.00 -> 4.44 mm
- net CS0: track 210.2 -> 213.2 mm
- net MOSI: track 209.2 -> 211.0 mm
- net EEPROM_WP: track 101.5 -> 103.2 mm
- net INT1_A: track 101.4 -> 102.6 mm
- net MISO: track 213.0 -> 213.9 mm
- net SDA: track 180.5 -> 181.3 mm
- net (no net): vias 0 -> 5
Other:
- board text added: "Encoder Board Blake Garner Rev A 13 Jul 2019"

Commit message: Small changes.
Other:
- outline, holes or cut-outs redrawn
