File: EncoderBoard/EncoderBoard.kicad_pcb (KiCad board)
At the start: 2 copper layers, 221 x 61 mm, 222 parts, among them SW1 Rotary_Encoder_Switch, SW10 SW_Push_LED_Red, SW11 SW_Push_LED_Blue, SW12 SW_Push_LED_Red, SW13 SW_Push_LED_Yellow, SW14 SW_Push_LED_Green, SW15 SW_Push_LED_Blue, SW2 Rotary_Encoder_Switch, SW3 Rotary_Encoder_Switch, SW4 Rotary_Encoder_Switch, SW5 Rotary_Encoder_Switch, SW6 Rotary_Encoder_Switch, SW7 Rotary_Encoder_Switch, SW8 Rotary_Encoder_Switch, SW9 Rotary_Encoder_Switch, U1 MCP23S17_SO, U10 Display_OLED_128x32_I2C, U11 Display_OLED_128x32_I2C, U12 Display_OLED_128x32_I2C, U13 Display_OLED_128x32_I2C, U14 Display_OLED_128x32_I2C, U15 Display_OLED_128x32_I2C, U16 Display_OLED_128x32_I2C, U17 Display_OLED_128x32_I2C, U18 74LVC14, U19 74LCV14, U2 MCP23S17_SO, U20 74LVC14, U21 74LVC14, U22 74LVC14, U23 74LVC14, U24 CAT24M01W, U25 CAT24M01W, U26 CAT24M01W, U3 MCP23S17_SO, U4 TCA9548APWR, U5 74HCT245, U6 TCA9548APWR, U7 Teensy3.2, U8 CAT24M01W, U9 Display_OLED_128x32_I2C

Commit message: Final revision of Rev A Board + Acrylic Case
Parts:
- R26, R38: value 120 -> 150
- R31, R51: value 68 -> 33
- U19: value 74LCV14 -> 74LVC14
Changed lines of the file:
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@@
   )
   (layers
-    (0 F.Cu signal hide)
-    (31 B.Cu signal hide)
-    (32 B.Adhes user hide)
+    (0 F.Cu signal)
+    (31 B.Cu signal)
+    (32 B.Adhes user)
     (33 F.Adhes user hide)
-    (34 B.Paste user hide)
+    (34 B.Paste user)
     (35 F.Paste user hide)
-    (36 B.SilkS user hide)
+    (36 B.SilkS user)
     (37 F.SilkS user)
-    (38 B.Mask user hide)
+    (38 B.Mask user)
     (39 F.Mask user)
     (40 Dwgs.User user)
@@
     (44 Edge.Cuts user)
     (45 Margin user)
-    (46 B.CrtYd user hide)
+    (46 B.CrtYd user)
     (47 F.CrtYd user hide)
-    (48 B.Fab user hide)
+    (48 B.Fab user)
     (49 F.Fab user)
   )
@@
     (solder_mask_min_width 0.05)
     (aux_axis_origin 0 0)
-    (visible_elements 7FF8FFBF)
+    (visible_elements 7FFFFFDF)
     (pcbplotparams
       (layerselection 0x010f0_ffffffff)
@@
       (effects (font (size 1 1) (thickness 0.15)))
     )
-    (fp_text value 120 (at 0 1.65) (layer F.Fab)
+    (fp_text value 150 (at 0 1.65) (layer F.Fab)
       (effects (font (size 1 1) (thickness 0.15)))
     )
@@
       (effects (font (size 1 1) (thickness 0.15)))
     )
-    (fp_text value 68 (at 0 1.65) (layer F.Fab)
+    (fp_text value 33 (at 0 1.65) (layer F.Fab)
       (effects (font (size 1 1) (thickness 0.15)))
     )
@@
       (effects (font (size 1 1) (thickness 0.15)))
     )
-    (fp_text value 120 (at 0 1.65 90) (layer F.Fab)
+    (fp_text value 150 (at 0 1.65 90) (layer F.Fab)
       (effects (font (size 1 1) (thickness 0.15)))
     )
@@
       (effects (font (size 1 1) (thickness 0.15)))
     )
-    (fp_text value 68 (at 0 1.65) (layer F.Fab)
+    (fp_text value 33 (at 0 1.65) (layer F.Fab)
       (effects (font (size 1 1) (thickness 0.15)))
     )
@@
     (tags resistor)
     (attr smd)
-    (fp_text reference R74 (at -3.25 2 90) (layer B.SilkS)
+    (fp_text reference R74 (at 0 -1.7 90) (layer B.SilkS)
       (effects (font (size 1 1) (thickness 0.15)) (justify mirror))
     )
@@
     (tags resistor)
     (attr smd)
-    (fp_text reference R79 (at 0 3.75 90) (layer B.SilkS)
+    (fp_text reference R79 (at 3.3 0 90) (layer B.SilkS)
       (effects (font (size 1 1) (thickness 0.15)) (justify mirror))
     )
@@
       (effects (font (size 1 1) (thickness 0.15)) (justify mirror))
     )
-    (fp_text value 10k (at 0 -3.5 90) (layer B.Fab)
+    (fp_text value 10k (at 3.1 0 90) (layer B.Fab)
       (effects (font (size 1 1) (thickness 0.15)) (justify mirror))
     )
@@
       (effects (font (size 1 1) (thickness 0.15)) (justify mirror))
     )
-    (fp_text value 10k (at -2.5 -2 90) (layer B.Fab)
+    (fp_text value 10k (at 0 1.6 90) (layer B.Fab)
       (effects (font (size 1 1) (thickness 0.15)) (justify mirror))
     )
@@
       (effects (font (size 1 1) (thickness 0.15)) (justify mirror))
     )
-    (fp_text value 74LCV14 (at 2.75 0.25 90) (layer B.Fab)
+    (fp_text value 74LVC14 (at 2.75 0.25 90) (layer B.Fab)
       (effects (font (size 1 1) (thickness 0.15)) (justify mirror))
     )
