File: EncoderBoard/Encoders&Buttons.sch (KiCad schematic (older format))
At the start: 73 parts

Commit message: Updated all switches to LED. Added EEPROM. Added rough costing.
Decided all switches could be LED (I can work out the colours later).
The EEPROM is a 1Mb model - might come in handy later.
Rough Costs was just to get a decent sense of how much this project will actually cost. Thankfully I already have some Pis...
Parts:
- removed SW? (x2): SW_Push, symbol Switch:SW_Push
- added R? (x2): R, symbol Device:R
- added SW? (x2): SW_Push_LED, symbol Switch:SW_Push_LED
Connections:
- net labels added: BUTTON0_LED, BUTTON1_LED
- wire segments 214 -> 220
Changed lines of the file:
@@
 	6600 4850 6500 4850
-$Comp
-L Switch:SW_Push SW?
-U 1 1 5D0B0E31
-P 9250 1700
-AR Path="/5D0B0E31" Ref="SW?"  Part="1"
-AR Path="/5CFF3BEB/5D0B0E31" Ref="SW?"  Part="1"
-F 0 "SW?" H 9250 1985 50  0000 C CNN
-F 1 "SW_Push" H 9250 1894 50  0000 C CNN
-F 2 "" H 9250 1900 50  0001 C CNN
-F 3 "~" H 9250 1900 50  0001 C CNN
-	1    9250 1700
-	1    0    0    -1
-$EndComp
 $Comp
 L Switch:SW_Push_LED SW?
@@
 	1    0    0    -1
 $EndComp
-$Comp
-L Switch:SW_Push SW?
-U 1 1 5D0B0E61
-P 9250 1150
-AR Path="/5D0B0E61" Ref="SW?"  Part="1"
-AR Path="/5CFF3BEB/5D0B0E61" Ref="SW?"  Part="1"
-F 0 "SW?" H 9250 1435 50  0000 C CNN
-F 1 "SW_Push" H 9250 1344 50  0000 C CNN
-F 2 "" H 9250 1350 50  0001 C CNN
-F 3 "~" H 9250 1350 50  0001 C CNN
-	1    9250 1150
-	1    0    0    -1
-$EndComp
-Text GLabel 9600 1150 2    50   Input ~ 0
+Text GLabel 9600 850  2    50   Input ~ 0
 BUTTON0_SW
-Text GLabel 9600 1700 2    50   Input ~ 0
+Text GLabel 9600 1550 2    50   Input ~ 0
 BUTTON1_SW
 Text GLabel 9600 2250 2    50   Input ~ 0
@@
 BUTTON5_SW
 Wire Wire Line
-	9600 1150 9450 1150
-Wire Wire Line
-	9600 1700 9450 1700
+	9600 850  9450 850
+Wire Wire Line
+	9600 1550 9450 1550
 Wire Wire Line
 	9600 2250 9450 2250
@@
 L power:GND #PWR?
 U 1 1 5D18CFA1
-P 8450 1800
+P 8450 1650
 AR Path="/5D18CFA1" Ref="#PWR?"  Part="1"
 AR Path="/5CFF3BEB/5D18CFA1" Ref="#PWR0209"  Part="1"
-F 0 "#PWR0209" H 8450 1550 50  0001 C CNN
-F 1 "GND" H 8455 1627 50  0000 C CNN
-F 2 "" H 8450 1800 50  0001 C CNN
-F 3 "" H 8450 1800 50  0001 C CNN
-	1    8450 1800
+F 0 "#PWR0209" H 8450 1400 50  0001 C CNN
+F 1 "GND" H 8455 1477 50  0000 C CNN
+F 2 "" H 8450 1650 50  0001 C CNN
+F 3 "" H 8450 1650 50  0001 C CNN
+	1    8450 1650
 	1    0    0    -1
 $EndComp
@@
 L power:GND #PWR?
 U 1 1 5D18D87A
-P 8450 1250
+P 8450 950
 AR Path="/5D18D87A" Ref="#PWR?"  Part="1"
 AR Path="/5CFF3BEB/5D18D87A" Ref="#PWR0210"  Part="1"
-F 0 "#PWR0210" H 8450 1000 50  0001 C CNN
-F 1 "GND" H 8455 1077 50  0000 C CNN
-F 2 "" H 8450 1250 50  0001 C CNN
-F 3 "" H 8450 1250 50  0001 C CNN
-	1    8450 1250
-	1    0    0    -1
-$EndComp
-Wire Wire Line
-	9050 1150 8450 1150
-Wire Wire Line
-	8450 1150 8450 1250
-Wire Wire Line
-	9050 1700 8450 1700
-Wire Wire Line
-	8450 1700 8450 1800
+F 0 "#PWR0210" H 8450 700 50  0001 C CNN
+F 1 "GND" H 8455 777 50  0000 C CNN
+F 2 "" H 8450 950 50  0001 C CNN
+F 3 "" H 8450 950 50  0001 C CNN
+	1    8450 950
+	1    0    0    -1
+$EndComp
+Wire Wire Line
+	9050 850  8450 850
+Wire Wire Line
+	8450 850  8450 950
+Wire Wire Line
+	9050 1550 8450 1550
+Wire Wire Line
+	8450 1550 8450 1650
 Wire Wire Line
 	8600 2350 8450 2350
@@
 Wire Wire Line
 	8450 2950 9050 2950
+$Comp
+L Switch:SW_Push_LED SW?
+U 1 1 5CF7287A
+P 9250 1650
+AR Path="/5CF7287A" Ref="SW?"  Part="1"
+AR Path="/5CFF3BEB/5CF7287A" Ref="SW?"  Part="1"
+F 0 "SW?" H 9250 2035 50  0000 C CNN
+F 1 "SW_Push_LED" H 9250 1944 50  0000 C CNN
+F 2 "" H 9250 1950 50  0001 C CNN
+F 3 "~" H 9250 1950 50  0001 C CNN
+	1    9250 1650
+	1    0    0    -1
+$EndComp
+$Comp
+L Switch:SW_Push_LED SW?
+U 1 1 5CF7337F
+P 9250 950
+AR Path="/5CF7337F" Ref="SW?"  Part="1"
+AR Path="/5CFF3BEB/5CF7337F" Ref="SW?"  Part="1"
+F 0 "SW?" H 9250 1335 50  0000 C CNN
+F 1 "SW_Push_LED" H 9250 1244 50  0000 C CNN
+F 2 "" H 9250 1250 50  0001 C CNN
+F 3 "~" H 9250 1250 50  0001 C CNN
+	1    9250 950
+	1    0    0    -1
+$EndComp
+Text GLabel 9600 1650 2    50   Input ~ 0
+BUTTON1_LED
+Wire Wire Line
+	9600 1650 9450 1650
+Text GLabel 9600 950  2    50   Input ~ 0
+BUTTON0_LED
+Wire Wire Line
+	9600 950  9450 950
+$Comp
+L Device:R R?
+U 1 1 5CF9FE26
+P 8750 1650
+F 0 "R?" V 8543 1650 50  0000 C CNN
+F 1 "R" V 8634 1650 50  0000 C CNN
+F 2 "" V 8680 1650 50  0001 C CNN
+F 3 "~" H 8750 1650 50  0001 C CNN
+	1    8750 1650
+	0    1    1    0
+$EndComp
+$Comp
+L Device:R R?
+U 1 1 5CFA080E
+P 8750 950
+F 0 "R?" V 8543 950 50  0000 C CNN
+F 1 "R" V 8634 950 50  0000 C CNN
+F 2 "" V 8680 950 50  0001 C CNN
+F 3 "~" H 8750 950 50  0001 C CNN
+	1    8750 950
+	0    1    1    0
+$EndComp
+Wire Wire Line
+	8900 950  9050 950
+Wire Wire Line
+	9050 1650 8900 1650
+Wire Wire Line
+	8600 1650 8450 1650
+Connection ~ 8450 1650
+Wire Wire Line
+	8600 950  8450 950
+Connection ~ 8450 950
 $EndSCHEMATC

Commit message: Updated schematic with appropriate symbols and latest library.
Parts:
- C? (x18): symbol Device:C -> Device:C_Small

Commit message: Generated draft footprint PCB with (very) approximate placements.
Parts:
- C12, C13, C14, C15, C16, C17, C18, C19, C20, C21, C22, C23, C24, C25, C26, C27, C28, C29: renamed from C?; footprint (none) -> Capacitor_BG:C_0805_2012Metric
- R22, R23, R24, R25, R27, R28, R29, R30, R32, R33, R34, R35, R36, R37, R39, R40, R42, R43, R44, R45, R46, R47, R49, R50, R52, R53, R54, R55, R56, R57, R58, R59, R60, R61, R62, R63: renamed from R?; footprint (none) -> Resistor_BG:R_0805_2012Metric
- R26, R38, R41, R48: renamed from R?; value R -> 120; footprint (none) -> Resistor_BG:R_0805_2012Metric
- R31, R51: renamed from R?; value R -> 68; footprint (none) -> Resistor_BG:R_0805_2012Metric
- SW1, SW2, SW3, SW4, SW5, SW6, SW7, SW8, SW9: renamed from SW?; footprint (none) -> Encoder_BG:RotaryEncoder_Bourns_PEC12R-4x20k-Sxxxx-Switch_Vertical_H20mm
- SW10: renamed from SW?; value SW_Push_LED -> SW_Push_LED_Red; footprint (none) -> Button_Switch_BG:E-Switch_SPST_Red_LED_RoundCap_TL3240F160R; symbol Switch:SW_Push_LED -> Switch_BG:SW_Push_LED
- SW11: renamed from SW?; value SW_Push_LED -> SW_Push_LED_Blue; footprint (none) -> Button_Switch_BG:E-Switch_SPST_LED_RoundCap_TL3240F160x; symbol Switch:SW_Push_LED -> Switch_BG:SW_Push_LED
- SW12: renamed from SW?; value SW_Push_LED -> SW_Push_LED_Red; footprint (none) -> Button_Switch_BG:E-Switch_SPST_Red_LED_SquareCap_TL3240F160R; symbol Switch:SW_Push_LED -> Switch_BG:SW_Push_LED
- SW13: renamed from SW?; value SW_Push_LED -> SW_Push_LED_Yellow; footprint (none) -> Button_Switch_BG:E-Switch_SPST_LED_SquareCap_TL3240F160x; symbol Switch:SW_Push_LED -> Switch_BG:SW_Push_LED
- SW14: renamed from SW?; value SW_Push_LED -> SW_Push_LED_Green; footprint (none) -> Button_Switch_BG:E-Switch_SPST_LED_SquareCap_TL3240F160x; symbol Switch:SW_Push_LED -> Switch_BG:SW_Push_LED
- SW15: renamed from SW?; value SW_Push_LED -> SW_Push_LED_Blue; footprint (none) -> Button_Switch_BG:E-Switch_SPST_LED_SquareCap_TL3240F160x; symbol Switch:SW_Push_LED -> Switch_BG:SW_Push_LED
Connections:
- wire segments 220 -> 217
- no-connect marks 0 -> 12
Other:
- moved on the sheet: R26, R31, R38, R41, R48, R51

Commit message: Tidied up the encoder board, updated debounce logic for schematic.
Parts:
- added C42, C43, C44, C48, C49, C50, C51, C55, C56: 0.01uF, Capacitor_BG:C_0805_2012Metric, symbol Device:C_Small
- added C45, C46, C47, C52, C53, C54, C57, C58, C59, C60, C61, C62: 0.1uF, Capacitor_BG:C_0805_2012Metric, symbol Device:C_Small
- added R64, R65, R66, R67, R68, R69, R70, R71, R72, R73, R74, R75, R76, R77, R78, R79, R80, R81, R82, R83, R84, R85, R86, R87: 10k, Resistor_BG:R_0805_2012Metric, symbol Device:R
- added U18, U19, U20, U21, U22, U23: 74LV14, symbol 74xx:74LV14
- C12, C13, C16, C17, C21, C22, C23, C24, C29: value 0.1uF -> 0.01uF
- R27, R28, R29, R30, R36, R37, R39, R40, R46, R47, R49, R50, R56, R57, R58, R59, R62, R63: value 1k -> 10k
Connections:
- net +3V3: now also R28.1, R30.1, R39.1, R40.1, R46.1, R56.1, R58.1, R59.1, C57.1, C58.1, C59.1, C60.1, C61.1, C62.1, R69.1, R70.1, R71.1, R73.1, R74.1, R75.1, R82.1, R83.1, R84.1, U18.14 (3.3V), U19.14 (3.3V), U20.14 (3.3V), U21.14 (3.3V), U22.14 (3.3V), U23.14 (3.3V); no longer R24.1, R33.1, R34.1, R35.1, R42.1, R52.1, R53.1, R54.1
- net BUTTON0_SW: now also U19.2; no longer SW10.3
- net BUTTON1_SW: now also U20.4; no longer SW11.3
- net BUTTON2_SW: now also U21.6; no longer SW12.3
- net BUTTON3_SW: now also U21.8; no longer SW13.3
- net BUTTON4_SW: now also U22.10; no longer SW14.3
- net BUTTON5_SW: now also U22.12; no longer SW15.3
- net ENC0_A: now also U18.2; no longer C12.1, R27.2
- net ENC0_B: now also U18.4; no longer C13.1, R29.2
- net ENC0_SW: now also U18.6; no longer SW1.S1
- net ENC1_A: now also U19.8; no longer C16.1, R36.2
- net ENC1_B: now also U19.10; no longer C17.1, R39.2
- net ENC1_SW: now also U19.12; no longer SW2.S1
- net ENC2_A: now also U21.2; no longer C20.1, R46.2
- net ENC2_B: now also U21.4; no longer C21.1, R49.2
- net ENC2_SW: now also U20.6; no longer SW3.S1
- net ENC3_A: now also U22.8; no longer C24.1, R56.2
- net ENC3_B: now also U21.10; no longer C25.1, R58.2
- net ENC3_SW: now also U21.12; no longer SW4.S1
- net ENC4_A: now also U23.2; no longer C28.1, R62.2
- net ENC4_B: now also U23.4; no longer C29.1, R63.2
- net ENC4_SW: now also U23.6; no longer SW5.S1
- net ENC5_A: now also U18.8; no longer C14.1, R28.2
- net ENC5_B: now also U18.10; no longer C15.1, R30.2
- net ENC5_SW: now also U18.12; no longer SW6.S1
- net ENC6_A: now also U20.2; no longer C18.1, R37.2
- net ENC6_B: now also U19.4; no longer C19.1, R40.2
- net ENC6_SW: now also U19.6; no longer SW7.S1
- net ENC7_A: now also U20.8; no longer C22.1, R47.2
- net ENC7_B: now also U20.10; no longer C23.1, R50.2
- net ENC7_SW: now also U20.12; no longer SW8.S1
- net ENC8_A: now also U22.2; no longer C26.1, R57.2
- net ENC8_B: now also U22.4; no longer C27.1, R59.2
- net ENC8_SW: now also U22.6; no longer SW9.S1
- net GND: now also C42.2, C43.2, C44.2, C45.2, C46.2, C47.2, C48.2, C49.2, C50.2, C51.2, C52.2, C53.2, C54.2, C55.2, C56.2, C57.2, C58.2, C59.2, C60.2, C61.2, C62.2, U18.7 (GND), U19.7 (GND), U20.7 (GND), U21.7 (GND), U22.7 (GND), U23.7 (GND)
- new net: R53.2, SW11.3
- new net: R36.2, SW10.3
- new net: R30.2, R33.2, SW1.S1
- new net: C12.1, R27.2, U18.1
- new net: C13.1, R29.2, U18.3
- new net: R37.1, R39.2, SW2.A
- new net: R40.2, R50.1, SW2.B
- new net: R45.2, R47.2, SW2.S1
- new net: R54.1, R55.2, SW3.A
- new net: R56.2, R65.1, SW3.B
- new net: R60.2, R62.2, SW3.S1
- new net: R68.1, R69.2, SW4.A
- new net: R70.2, R78.1, SW4.B
- new net: R71.2, R76.2, SW4.S1
- new net: R81.1, R82.2, SW5.A
- new net: R83.2, R87.1, SW5.B
- new net: R84.2, R85.2, SW5.S1
- new net: R24.1, R25.2, SW6.A
- new net: R28.2, R35.1, SW6.B
- new net: R32.2, R34.2, SW6.S1
- new net: R42.1, R43.2, SW7.A
- new net: R44.2, R52.1, SW7.B
- new net: R46.2, R49.2, SW7.S1
- new net: R57.1, R58.2, SW8.A
- new net: R59.2, R66.1, SW8.B
- new net: R61.2, R63.2, SW8.S1
- new net: R72.1, R73.2, SW9.A
- new net: R74.2, R79.1, SW9.B
- new net: R75.2, R77.2, SW9.S1
- new net: R64.2, SW12.3
- new net: R67.2, SW13.3
- new net: R80.2, SW14.3
- new net: R86.2, SW15.3
- new net: C14.1, R33.1, U18.5
- new net: C18.1, R36.1, U19.1
- new net: C25.1, R53.1, U20.3
- new net: C28.1, R64.1, U21.5
- new net: C45.1, R67.1, U21.9
- new net: C52.1, R80.1, U22.11
- new net: C54.1, R86.1, U22.13
- new net: C21.1, R37.2, U19.9
- new net: C22.1, R50.2, U19.11
- new net: C19.1, R47.1, U19.13
- new net: C29.1, R54.2, U21.1
- new net: C42.1, R65.2, U21.3
- new net: C48.1, R68.2, U22.9
- new net: C49.1, R78.2, U21.11
- new net: C55.1, R81.2, U23.1
- new net: C56.1, R87.2, U23.3
- new net: C16.1, R24.2, U18.9
- new net: C17.1, R35.2, U18.11
- new net: C26.1, R62.1, U20.5
- new net: C46.1, R76.1, U21.13
- new net: C53.1, R85.1, U23.5
- new net: C15.1, R34.1, U18.13
- new net: C23.1, R42.2, U20.1
- new net: C24.1, R52.2, U19.3
- new net: C43.1, R57.2, U20.9
- new net: C44.1, R66.2, U20.11
- new net: C50.1, R72.2, U22.1
- new net: C51.1, R79.2, U22.3
- new net: C20.1, R49.1, U19.5
- new net: C27.1, R63.1, U20.13
- new net: C47.1, R77.1, U22.5
Other:
- moved on the sheet: C12, C13, R22, R23, R26, R27, R29, R31, R38, R41, R48, R51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

Commit message: Completed final drafting of Encoder Board.
Not quite submitted yet - but pretty close to the final layout for the board to be made.
Parts:
- SW1, SW2, SW3, SW4, SW5, SW6, SW7, SW8, SW9: symbol Device:Rotary_Encoder_Switch -> Switch_BG:Rotary_Encoder_Switch
- U18, U20, U21, U22, U23: value 74LV14 -> 74LVC14; footprint (none) -> SOIC_BG:SOIC-14_3.9x8.7mm_P1.27mm
- U19: value 74LV14 -> 74LCV14; footprint (none) -> SOIC_BG:SOIC-14_3.9x8.7mm_P1.27mm
- U23: renamed from U22; value 74LV14 -> 74LVC14; footprint (none) -> SOIC_BG:SOIC-14_3.9x8.7mm_P1.27mm
Connections:
- net BUTTON0_SW: now also U22.2; no longer U19.2
- net BUTTON1_SW: now also U22.4; no longer U20.4
- net BUTTON2_SW: now also U23.2; no longer U21.6
- net BUTTON3_SW: now also U23.4; no longer U21.8
- net BUTTON4_SW: now also U23.6; no longer U22.10
- net BUTTON5_SW: now also U23.8; no longer U22.12
- net ENC0_A: now also U18.10; no longer U18.2
- net ENC0_B: now also U18.8; no longer U18.4
- net ENC0_SW: now also U18.12; no longer U18.6
- net ENC1_A: now also U18.6; no longer U19.8
- net ENC1_B: now also U18.4; no longer U19.10
- net ENC1_SW: now also U18.2; no longer U19.12
- net ENC2_A: now also U19.10; no longer U21.2
- net ENC2_B: now also U19.8; no longer U21.4
- net ENC2_SW: now also U19.12; no longer U20.6
- net ENC3_A: now also U19.6; no longer U22.8
- net ENC3_B: now also U19.4; no longer U21.10
- net ENC3_SW: now also U19.2; no longer U21.12
- net ENC4_A: now also U20.10; no longer U23.2
- net ENC4_B: now also U20.8; no longer U23.4
- net ENC4_SW: now also U20.12; no longer U23.6
- net ENC5_A: now also U20.6; no longer U18.8
- net ENC5_B: now also U20.4; no longer U18.10
- net ENC5_SW: now also U20.2; no longer U18.12
- net ENC6_A: now also U21.10; no longer U20.2
- net ENC6_B: now also U21.8; no longer U19.4
- net ENC6_SW: now also U21.12; no longer U19.6
- net ENC7_A: now also U21.6; no longer U20.8
- net ENC7_B: now also U21.4; no longer U20.10
- net ENC7_SW: now also U21.2; no longer U20.12
- net ENC8_A: now also U22.10; no longer U22.2
- net ENC8_B: now also U22.8; no longer U22.4
- net ENC8_SW: now also U22.12; no longer U23.6
- net GND: now also SW1.MP (Mounting_Point), SW2.MP (Mounting_Point), SW3.MP (Mounting_Point), SW4.MP (Mounting_Point), SW5.MP (Mounting_Point), SW6.MP (Mounting_Point), SW7.MP (Mounting_Point), SW8.MP (Mounting_Point), SW9.MP (Mounting_Point)
- net at C12.1, R27.2: now also U18.11; no longer U18.1
- net at C13.1, R29.2: now also U18.9; no longer U18.3
- net at C14.1, R33.1: now also U18.13; no longer U18.5
- net at C18.1, R36.1: now also U22.1; no longer U19.1
- net at C25.1, R53.1: now also U22.3; no longer U20.3
- net at C28.1, R64.1: now also U23.1; no longer U21.5
- net at C45.1, R67.1: now also U23.3; no longer U21.9
- net at C52.1, R80.1: now also U23.5; no longer U22.11
- net at C54.1, R86.1: now also U23.9; no longer U22.13
- net at C21.1, R37.2: now also U18.5; no longer U19.9
- net at C22.1, R50.2: now also U18.3; no longer U19.11
- net at C19.1, R47.1: now also U18.1; no longer U19.13
- net at C29.1, R54.2: now also U19.11; no longer U21.1
- net at C42.1, R65.2: now also U19.9; no longer U21.3
- net at C48.1, R68.2: now also U19.5; no longer U22.9
- net at C49.1, R78.2: now also U19.3; no longer U21.11
- net at C55.1, R81.2: now also U20.11; no longer U23.1
- net at C56.1, R87.2: now also U20.9; no longer U23.3
- net at C16.1, R24.2: now also U20.5; no longer U18.9
- net at C17.1, R35.2: now also U20.3; no longer U18.11
- net at C26.1, R62.1: now also U19.13; no longer U20.5
- net at C46.1, R76.1: now also U19.1; no longer U21.13
- net at C53.1, R85.1: now also U20.13; no longer U23.5
- net at C15.1, R34.1: now also U20.1; no longer U18.13
- net at C23.1, R42.2: now also U21.11; no longer U20.1
- net at C24.1, R52.2: now also U21.9; no longer U19.3
- net at C43.1, R57.2: now also U21.5; no longer U20.9
- net at C44.1, R66.2: now also U21.3; no longer U20.11
- net at C50.1, R72.2: now also U22.11; no longer U22.1
- net at C51.1, R79.2: now also U22.9; no longer U22.3
- net at C20.1, R49.1: now also U21.13; no longer U19.5
- net at C27.1, R63.1: now also U21.1; no longer U20.13
- net at C47.1, R77.1: now also U22.13; no longer U23.5
Other:
- moved on the sheet: U18A, U18B, U18C, U18D, U18E, U18F, U19A, U19B, U19C, U19D, U19E, U19F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

Commit message: Final version of Rev A board.
- Fixed up address pins on some chips.
- Added some additional bypass capacitors.
- Fixed up some broken footprint references.
- Some minor layout adjustments.
Parts:
- C12, C13, C16, C17, C21, C22, C23, C24, C29, C42, C43, C44, C48, C49, C50, C51, C55, C56: value 0.01uF -> 10nF
- C14, C15, C18, C19, C20, C25, C26, C27, C28, C45, C46, C47, C52, C53, C54, C57, C58, C59, C60, C61, C62: value 0.1uF -> 100nF

Commit message: Small changes.
Parts:
- R26, R38: value 120 -> 150
- R31, R51: value 68 -> 33
Changed lines of the file:
@@
 EESchema Schematic File Version 4
-LIBS:EncoderBoard-cache
 EELAYER 29 0
 EELAYER END
 $Descr A4 11693 8268
 encoding utf-8
-Sheet 2 3
+Sheet 1 1
 Title "Encoder Board"
 Date "2019-07-15"
@@
 P 8350 3900
 F 0 "R38" V 8143 3900 50  0000 C CNN
-F 1 "120" V 8234 3900 50  0000 C CNN
+F 1 "150" V 8234 3900 50  0000 C CNN
 F 2 "Resistor_BG:R_0805_2012Metric" V 8280 3900 50  0001 C CNN
 F 3 "~" H 8350 3900 50  0001 C CNN
@@
 P 8350 6250
 F 0 "R51" V 8143 6250 50  0000 C CNN
-F 1 "68" V 8234 6250 50  0000 C CNN
+F 1 "33" V 8234 6250 50  0000 C CNN
 F 2 "Resistor_BG:R_0805_2012Metric" V 8280 6250 50  0001 C CNN
 F 3 "~" H 8350 6250 50  0001 C CNN
@@
 P 8350 2950
 F 0 "R31" V 8143 2950 50  0000 C CNN
-F 1 "68" V 8234 2950 50  0000 C CNN
+F 1 "33" V 8234 2950 50  0000 C CNN
 F 2 "Resistor_BG:R_0805_2012Metric" V 8280 2950 50  0001 C CNN
 F 3 "~" H 8350 2950 50  0001 C CNN
@@
 P 8350 1700
 F 0 "R26" V 8143 1700 50  0000 C CNN
-F 1 "120" V 8234 1700 50  0000 C CNN
+F 1 "150" V 8234 1700 50  0000 C CNN
 F 2 "Resistor_BG:R_0805_2012Metric" V 8280 1700 50  0001 C CNN
 F 3 "~" H 8350 1700 50  0001 C CNN

Commit message: Final revision of Rev A Board + Acrylic Case
Parts:
- U19: value 74LCV14 -> 74LVC14
Changed lines of the file:
@@
 EESchema Schematic File Version 4
+LIBS:EncoderBoard-cache
 EELAYER 29 0
 EELAYER END
 $Descr A4 11693 8268
 encoding utf-8
-Sheet 1 1
+Sheet 2 3
 Title "Encoder Board"
 Date "2019-07-15"
@@
 P 1150 3800
 F 0 "U19" H 1250 3550 50  0000 C CNN
-F 1 "74LCV14" H 1250 3650 50  0000 C CNN
+F 1 "74LVC14" H 1250 3650 50  0000 C CNN
 F 2 "SOIC_BG:SOIC-14_3.9x8.7mm_P1.27mm" H 1150 3800 50  0001 C CNN
 F 3 "http://www.ti.com/lit/gpn/sn74LV14" H 1150 3800 50  0001 C CNN
@@
 P 1150 3400
 F 0 "U19" H 1250 3150 50  0000 C CNN
-F 1 "74LCV14" H 1250 3250 50  0000 C CNN
+F 1 "74LVC14" H 1250 3250 50  0000 C CNN
 F 2 "SOIC_BG:SOIC-14_3.9x8.7mm_P1.27mm" H 1150 3400 50  0001 C CNN
 F 3 "http://www.ti.com/lit/gpn/sn74LV14" H 1150 3400 50  0001 C CNN
@@
 P 3850 3600
 F 0 "U19" H 3950 3850 50  0000 C CNN
-F 1 "74LCV14" H 3950 3750 50  0000 C CNN
+F 1 "74LVC14" H 3950 3750 50  0000 C CNN
 F 2 "SOIC_BG:SOIC-14_3.9x8.7mm_P1.27mm" H 3850 3600 50  0001 C CNN
 F 3 "http://www.ti.com/lit/gpn/sn74LV14" H 3850 3600 50  0001 C CNN
@@
 U 2 1 5D8B821B
 P 10350 4400
-F 0 "U23" H 10500 4600 50  0000 C CNN
+F 0 "U23" H 10500 4650 50  0000 C CNN
 F 1 "74LVC14" H 10500 4550 50  0000 C CNN
 F 2 "SOIC_BG:SOIC-14_3.9x8.7mm_P1.27mm" H 10350 4400 50  0001 C CNN
@@
 P 1150 5000
 F 0 "U19" H 1250 4750 50  0000 C CNN
-F 1 "74LCV14" H 1250 4850 50  0000 C CNN
+F 1 "74LVC14" H 1250 4850 50  0000 C CNN
 F 2 "SOIC_BG:SOIC-14_3.9x8.7mm_P1.27mm" H 1150 5000 50  0001 C CNN
 F 3 "http://www.ti.com/lit/gpn/sn74LV14" H 1150 5000 50  0001 C CNN
@@
 P 1150 4600
 F 0 "U19" H 1250 4350 50  0000 C CNN
-F 1 "74LCV14" H 1250 4450 50  0000 C CNN
+F 1 "74LVC14" H 1250 4450 50  0000 C CNN
 F 2 "SOIC_BG:SOIC-14_3.9x8.7mm_P1.27mm" H 1150 4600 50  0001 C CNN
 F 3 "http://www.ti.com/lit/gpn/sn74LV14" H 1150 4600 50  0001 C CNN
@@
 P 3850 4800
 F 0 "U19" H 4000 5050 50  0000 C CNN
-F 1 "74LCV14" H 4000 4950 50  0000 C CNN
+F 1 "74LVC14" H 4000 4950 50  0000 C CNN
 F 2 "SOIC_BG:SOIC-14_3.9x8.7mm_P1.27mm" H 3850 4800 50  0001 C CNN
 F 3 "http://www.ti.com/lit/gpn/sn74LV14" H 3850 4800 50  0001 C CNN
@@
 P 3150 7100
 F 0 "U19" H 3450 7150 50  0000 L CNN
-F 1 "74LCV14" H 3450 7050 50  0000 L CNN
+F 1 "74LVC14" H 3450 7050 50  0000 L CNN
 F 2 "SOIC_BG:SOIC-14_3.9x8.7mm_P1.27mm" H 3150 7100 50  0001 C CNN
 F 3 "http://www.ti.com/lit/gpn/sn74LV14" H 3150 7100 50  0001 C CNN
