File: Hardware/EncoderBoard.kicad_pcb (KiCad board)
At the start: 2 copper layers, 221 x 61 mm, 222 parts, among them SW1 Rotary_Encoder_Switch, SW10 SW_Push_LED_Red, SW11 SW_Push_LED_Blue, SW12 SW_Push_LED_Red, SW13 SW_Push_LED_Yellow, SW14 SW_Push_LED_Green, SW15 SW_Push_LED_Blue, SW2 Rotary_Encoder_Switch, SW3 Rotary_Encoder_Switch, SW4 Rotary_Encoder_Switch, SW5 Rotary_Encoder_Switch, SW6 Rotary_Encoder_Switch, SW7 Rotary_Encoder_Switch, SW8 Rotary_Encoder_Switch, SW9 Rotary_Encoder_Switch, U1 MCP23S17_SO, U10 Display_OLED_128x32_I2C, U11 Display_OLED_128x32_I2C, U12 Display_OLED_128x32_I2C, U13 Display_OLED_128x32_I2C, U14 Display_OLED_128x32_I2C, U15 Display_OLED_128x32_I2C, U16 Display_OLED_128x32_I2C, U17 Display_OLED_128x32_I2C, U18 74LVC14, U19 74LVC14, U2 MCP23S17_SO, U20 74LVC14, U21 74LVC14, U22 74LVC14, U23 74LVC14, U24 CAT24M01W, U25 CAT24M01W, U26 CAT24M01W, U3 MCP23S17_SO, U4 TCA9548APWR, U5 74HCT245, U6 TCA9548APWR, U7 Teensy3.2, U8 CAT24M01W, U9 Display_OLED_128x32_I2C

Commit message: Fixed missing pull-up resistors and published RevB of PCB.
Parts:
- added R90: 10k, Resistor_BG:R_0805_2012Metric, F.Cu at (266.7, 83.2)
- added R91: 10k, Resistor_BG:R_0805_2012Metric, F.Cu at (225.9, 68.5)
- added R92: 10k, Resistor_BG:R_0805_2012Metric, F.Cu at (62.6, 58.9)
- added R93: 10k, Resistor_BG:R_0805_2012Metric, F.Cu at (62.9, 73.0)
- added R94: 10k, Resistor_BG:R_0805_2012Metric, F.Cu at (62.6, 87.0)
- added R95: 10k, Resistor_BG:R_0805_2012Metric, F.Cu at (62.5, 101.0)
Routing:
- net +3V3: track 1021.8 -> 1074.6 mm, vias 19 -> 24
- net Net-(C45-Pad1): track 242.2 -> 248.6 mm
- net Net-(R53-Pad2): track 6.41 -> 9.78 mm
- net Net-(C25-Pad1): track 35.9 -> 38.2 mm
- net Net-(R64-Pad2): track 2.54 -> 3.97 mm
- net Net-(R67-Pad2): track 2.37 -> 3.79 mm
- net Net-(R80-Pad2): track 2.54 -> 3.91 mm
- net Net-(R86-Pad2): track 4.83 -> 6.13 mm
- net GND: track 711.1 -> 711.8 mm
Other:
- board text added: "Encoder Board Blake Garner Rev B 2 Jun 2020"
- board text removed: "Encoder Board Blake Garner Rev A 13 Jul 2019"
