File: Hardware/EncoderBoard.kicad_pcb (KiCad board)
At the start: 2 copper layers, 221 x 61 mm, 228 parts, among them SW1 Rotary_Encoder_Switch, SW10 SW_Push_LED_Red, SW11 SW_Push_LED_Blue, SW12 SW_Push_LED_Red, SW13 SW_Push_LED_Yellow, SW14 SW_Push_LED_Green, SW15 SW_Push_LED_Blue, SW2 Rotary_Encoder_Switch, SW3 Rotary_Encoder_Switch, SW4 Rotary_Encoder_Switch, SW5 Rotary_Encoder_Switch, SW6 Rotary_Encoder_Switch, SW7 Rotary_Encoder_Switch, SW8 Rotary_Encoder_Switch, SW9 Rotary_Encoder_Switch, U1 MCP23S17_SO, U10 Display_OLED_128x32_I2C, U11 Display_OLED_128x32_I2C, U12 Display_OLED_128x32_I2C, U13 Display_OLED_128x32_I2C, U14 Display_OLED_128x32_I2C, U15 Display_OLED_128x32_I2C, U16 Display_OLED_128x32_I2C, U17 Display_OLED_128x32_I2C, U18 74LVC14, U19 74LVC14, U2 MCP23S17_SO, U20 74LVC14, U21 74LVC14, U22 74LVC14, U23 74LVC14, U24 CAT24M01W, U25 CAT24M01W, U26 CAT24M01W, U3 MCP23S17_SO, U4 TCA9548APWR, U5 74HCT245, U6 TCA9548APWR, U7 Teensy3.2, U8 CAT24M01W, U9 Display_OLED_128x32_I2C

Commit message: Applied MPN to each item and consolidated some parts
Parts:
- added R96: 150R, Resistor_BG:R_0805_2012Metric, F.Cu at (239.9, 71.5)
- C1, C10, C14, C15, C18, C19, C20, C25, C26, C27, C28, C3, C30, C31, C32, C33, C34, C35, C36, C37, C38, C39, C40, C41, C45, C46, C47, C5, C52, C53, C54, C57, C58, C59, C60, C61, C62, C63, C64, C65, C66, C67, C68, C69, C7, C70, C71, C72, C73, C74, C75, C9: value 100nF -> 0.1uF
- C12, C13, C16, C17, C21, C22, C23, C24, C29, C42, C43, C44, C48, C49, C50, C51, C55, C56: value 10nF -> 0.01uF
- R17: value 330R -> 150R
- R26, R38: value 150 -> 150R
- R31, R51: value 33 -> 33R
- R41, R48: value 120 -> 150R
- SW1, SW2, SW3, SW4, SW5, SW6, SW7, SW8, SW9: value Rotary_Encoder_Switch -> Encoder_SW_D12.0xH25.0mm
- moved R17 3.06 mm to (236.7, 71.5)
Connections:
- R17 pad 1: WS2812_DATA -> Net-(R17-Pad1)
Routing:
- net /WS2812_3V3: track 51.6 -> 59.8 mm
- net +5V: track 567.3 -> 565.5 mm
- net Net-(R17-Pad2): track 3.49 -> 5.00 mm
- net Net-(R17-Pad1): track 0.00 -> 1.27 mm
- net GND: track 711.8 -> 711.2 mm

Commit message: Finished (untested) sketch of the Rev C PCB.
TODO: Revise svg, 3D model and PDFs of the acrylic.
Parts:
- removed REF** (x5): MountingHole_3.2mm_M3, MountingHole:MountingHole_3.2mm_M3
- added ?: M3_Hole, MountingHole:MountingHole_3.2mm_M3, F.Cu at (142.0, 66.5)
- added ?: M3_Hole, MountingHole:MountingHole_3.2mm_M3, F.Cu at (23.5, 23.5)
- added ?: M3_Hole, MountingHole:MountingHole_3.2mm_M3, F.Cu at (248.0, 23.5)
- added ?: M3_Hole, MountingHole:MountingHole_3.2mm_M3, F.Cu at (248.0, 81.5)
- added ?: M3_Hole, MountingHole:MountingHole_3.2mm_M3, F.Cu at (143.0, 23.5)
- added ?: M3_Hole, MountingHole:MountingHole_3.2mm_M3, F.Cu at (23.5, 81.5)
- C18, C25, C28, C30, C31, C32, C45, C52, C54, C9, R17, R26, R36, R38, R41, R48, R53, R64, R67, R80, R86, R90, R91, R92, R93, R94, R95, R96, U5: moved to B.Cu
- R31, R51: value 33R -> 150R; moved to B.Cu
- SW10: footprint Button_Switch_BG:E-Switch_SPST_Red_LED_RoundCap_TL3240F160R -> Button_Switch_BG:TE_Alcoswitch_SPST_LED
- SW11: footprint Button_Switch_BG:E-Switch_SPST_LED_RoundCap_TL3240F160x -> Button_Switch_BG:TE_Alcoswitch_SPST_LED
- SW12: footprint Button_Switch_BG:E-Switch_SPST_Red_LED_SquareCap_TL3240F160R -> Button_Switch_BG:TE_Alcoswitch_SPST_LED
- SW13, SW14, SW15: footprint Button_Switch_BG:E-Switch_SPST_LED_SquareCap_TL3240F160x -> Button_Switch_BG:TE_Alcoswitch_SPST_LED
- moved C30 57.6 mm to (225.0, 26.0), turned to 180 degrees
- moved C31 57.1 mm to (233.0, 26.0), turned to 180 degrees
- moved C32 56.7 mm to (241.0, 26.0), turned to 180 degrees
- moved D1 55.5 mm to (223.0, 24.5), turned to 180 degrees
- moved D2 54.9 mm to (231.0, 24.5), turned to 180 degrees
- moved D3 54.3 mm to (239.0, 24.5), turned to 180 degrees
- moved U23 51.9 mm to (210.5, 76.5)
- moved C62 50.5 mm to (209.0, 70.5), turned to 0 degrees
- moved R17 48.8 mm to (205.0, 34.5)
- moved R96 48.5 mm to (208.5, 34.5)
- moved C73 46.8 mm to (186.5, 32.5)
- moved R86 46.7 mm to (32.0, 72.0), turned to 180 degrees
- moved R80 46.0 mm to (32.0, 59.0), turned to 180 degrees
- moved C75 45.8 mm to (186.5, 46.5)
- moved R41 45.8 mm to (28.5, 50.5)
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Connections:
- SW10 pad 2: (no net) -> GND
- SW10 pad 4: (no net) -> Net-(R36-Pad2)
- SW11 pad 2: (no net) -> GND
- SW11 pad 4: (no net) -> Net-(R53-Pad2)
- SW12 pad 2: (no net) -> GND
- SW12 pad 4: (no net) -> Net-(R64-Pad2)
- SW13 pad 2: (no net) -> GND
- SW13 pad 4: (no net) -> Net-(R67-Pad2)
- SW14 pad 2: (no net) -> GND
- SW14 pad 4: (no net) -> Net-(R80-Pad2)
- SW15 pad 2: (no net) -> GND
- SW15 pad 4: (no net) -> Net-(R86-Pad2)
Routing:
- net GND: track 711.2 -> 2263.1 mm, vias 38 -> 54
- net +3V3: track 1074.6 -> 1238.3 mm, vias 24 -> 41
- net BUTTON2_LED: track 223.0 -> 316.9 mm, vias 0 -> 2
- net SDA: track 181.3 -> 273.5 mm, vias 2 -> 3
- net SCL: track 196.0 -> 280.4 mm, vias 2 -> 3
- net +5V: track 565.5 -> 484.6 mm, vias 6 -> 13
- net Net-(D3-Pad2): track 19.1 -> 87.7 mm, vias 0 -> 2
- net BUTTON3_LED: track 231.9 -> 296.7 mm, vias 0 -> 2
- net Net-(C18-Pad1): track 31.5 -> 62.7 mm, vias 1 -> 2
- net BUTTON4_LED: track 249.4 -> 280.1 mm, vias 0 -> 1
- net Net-(C28-Pad1): track 243.4 -> 268.5 mm, vias 1 -> 2
- net SDA2: track 39.3 -> 62.5 mm
- net SCL2: track 33.8 -> 57.0 mm
- net BUTTON0_SW: track 14.5 -> 36.4 mm
- net BUTTON1_SW: track 14.9 -> 34.3 mm
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Other:
- board size 221 x 61 mm -> 231.5 x 65 mm
- net class Default: trace_width 0.3048 -> 0.254; via_dia 0.762 -> 1; via_drill 0.381 -> 0.6
- net class Power_3V3: trace_width 0.762 -> 0.508; via_dia 1.524 -> 1; via_drill 0.762 -> 0.6
- net class Power_5V: trace_width 1.016 -> 0.762; via_dia 1.524 -> 1; via_drill 0.762 -> 0.6
- rule solder_mask_min_width: 0.05 -> 0.15
- rule trace_min: 0.254 -> 0.1524
- board text added: "Encoder Board Blake Garner Rev C 10 Jun 2020"
- board text added: "Encoders for Eos Designed by Blake Garner"
- board text removed: "Encoder Board Blake Garner Rev B 2 Jun 2020"
