File: Hardware/EncoderBoard.kicad_pcb (KiCad board)
At the start: 2 copper layers, 231.5 x 65 mm, 230 parts, among them SW1 Encoder_SW_D12.0xH25.0mm, SW10 SW_Push_LED_Red, SW11 SW_Push_LED_Blue, SW12 SW_Push_LED_Red, SW13 SW_Push_LED_Yellow, SW14 SW_Push_LED_Green, SW15 SW_Push_LED_Blue, SW2 Encoder_SW_D12.0xH25.0mm, SW3 Encoder_SW_D12.0xH25.0mm, SW4 Encoder_SW_D12.0xH25.0mm, SW5 Encoder_SW_D12.0xH25.0mm, SW6 Encoder_SW_D12.0xH25.0mm, SW7 Encoder_SW_D12.0xH25.0mm, SW8 Encoder_SW_D12.0xH25.0mm, SW9 Encoder_SW_D12.0xH25.0mm, U1 MCP23S17_SO, U10 Display_OLED_128x32_I2C, U11 Display_OLED_128x32_I2C, U12 Display_OLED_128x32_I2C, U13 Display_OLED_128x32_I2C, U14 Display_OLED_128x32_I2C, U15 Display_OLED_128x32_I2C, U16 Display_OLED_128x32_I2C, U17 Display_OLED_128x32_I2C, U18 74LVC14, U19 74LVC14, U2 MCP23S17_SO, U20 74LVC14, U21 74LVC14, U22 74LVC14, U23 74LVC14, U24 CAT24M01W, U25 CAT24M01W, U26 CAT24M01W, U3 MCP23S17_SO, U4 TCA9548APWR, U5 74HCT245, U6 TCA9548APWR, U7 Teensy3.2, U8 CAT24M01W, U9 Display_OLED_128x32_I2C

Commit message: Updated acrylic cutouts for encoder board hardware
Other:
- board text added: "Encodie"
- board text removed: "Encoders for Eos Designed by Blake Garner"
