File: Hardware/Encoders&Buttons.sch (KiCad schematic (older format))
At the start: 126 parts, among them SW1 Rotary_Encoder_Switch, SW10 SW_Push_LED_Red, SW11 SW_Push_LED_Blue, SW12 SW_Push_LED_Red, SW13 SW_Push_LED_Yellow, SW14 SW_Push_LED_Green, SW15 SW_Push_LED_Blue, SW2 Rotary_Encoder_Switch, SW3 Rotary_Encoder_Switch, SW4 Rotary_Encoder_Switch, SW5 Rotary_Encoder_Switch, SW6 Rotary_Encoder_Switch, SW7 Rotary_Encoder_Switch, SW8 Rotary_Encoder_Switch, SW9 Rotary_Encoder_Switch, U18 74LVC14, U19 74LVC14, U20 74LVC14, U21 74LVC14, U22 74LVC14, U23 74LVC14

Commit message: Fixed missing pull-up resistors and published RevB of PCB.
Parts:
- added R90, R91, R92, R93, R94, R95: 10k, Resistor_BG:R_0805_2012Metric, symbol Device:R
Connections:
- net +3V3: now also R90.1, R91.1, R92.1, R93.1, R94.1, R95.1
- net at R53.2, SW11.3: now also R91.2
- net at R36.2, SW10.3: now also R90.2
- net at R64.2, SW12.3: now also R92.2
- net at R67.2, SW13.3: now also R93.2
- net at R80.2, SW14.3: now also R94.2
- net at R86.2, SW15.3: now also R95.2
Changed lines of the file:
@@
 	1    0    0    -1
 $EndComp
+$Comp
+L power:+3V3 #PWR0184
+U 1 1 5ED82242
+P 9550 1200
+F 0 "#PWR0184" H 9550 1050 50  0001 C CNN
+F 1 "+3V3" H 9565 1373 50  0000 C CNN
+F 2 "" H 9550 1200 50  0001 C CNN
+F 3 "" H 9550 1200 50  0001 C CNN
+	1    9550 1200
+	1    0    0    -1
+$EndComp
+$Comp
+L Device:R R?
+U 1 1 5ED81C21
+P 9550 1350
+AR Path="/5ED81C21" Ref="R?"  Part="1"
+AR Path="/5CFF3BEB/5ED81C21" Ref="R90"  Part="1"
+F 0 "R90" H 9500 1400 50  0000 R CNN
+F 1 "10k" H 9500 1300 50  0000 R CNN
+F 2 "Resistor_BG:R_0805_2012Metric" V 9480 1350 50  0001 C CNN
+F 3 "~" H 9550 1350 50  0001 C CNN
+	1    9550 1350
+	1    0    0    -1
+$EndComp
+$Comp
+L Device:R R?
+U 1 1 5EDF6647
+P 9550 2600
+AR Path="/5EDF6647" Ref="R?"  Part="1"
+AR Path="/5CFF3BEB/5EDF6647" Ref="R91"  Part="1"
+F 0 "R91" H 9500 2650 50  0000 R CNN
+F 1 "10k" H 9500 2550 50  0000 R CNN
+F 2 "Resistor_BG:R_0805_2012Metric" V 9480 2600 50  0001 C CNN
+F 3 "~" H 9550 2600 50  0001 C CNN
+	1    9550 2600
+	1    0    0    -1
+$EndComp
+$Comp
+L power:+3V3 #PWR0185
+U 1 1 5EDF664D
+P 9550 2450
+F 0 "#PWR0185" H 9550 2300 50  0001 C CNN
+F 1 "+3V3" H 9565 2623 50  0000 C CNN
+F 2 "" H 9550 2450 50  0001 C CNN
+F 3 "" H 9550 2450 50  0001 C CNN
+	1    9550 2450
+	1    0    0    -1
+$EndComp
+$Comp
+L Device:R R?
+U 1 1 5EE058ED
+P 9550 3550
+AR Path="/5EE058ED" Ref="R?"  Part="1"
+AR Path="/5CFF3BEB/5EE058ED" Ref="R92"  Part="1"
+F 0 "R92" H 9500 3600 50  0000 R CNN
+F 1 "10k" H 9500 3500 50  0000 R CNN
+F 2 "Resistor_BG:R_0805_2012Metric" V 9480 3550 50  0001 C CNN
+F 3 "~" H 9550 3550 50  0001 C CNN
+	1    9550 3550
+	1    0    0    -1
+$EndComp
+$Comp
+L power:+3V3 #PWR0186
+U 1 1 5EE058F3
+P 9550 3400
+F 0 "#PWR0186" H 9550 3250 50  0001 C CNN
+F 1 "+3V3" H 9565 3573 50  0000 C CNN
+F 2 "" H 9550 3400 50  0001 C CNN
+F 3 "" H 9550 3400 50  0001 C CNN
+	1    9550 3400
+	1    0    0    -1
+$EndComp
+$Comp
+L Device:R R?
+U 1 1 5EE14C5D
+P 9550 4250
+AR Path="/5EE14C5D" Ref="R?"  Part="1"
+AR Path="/5CFF3BEB/5EE14C5D" Ref="R93"  Part="1"
+F 0 "R93" H 9500 4300 50  0000 R CNN
+F 1 "10k" H 9500 4200 50  0000 R CNN
+F 2 "Resistor_BG:R_0805_2012Metric" V 9480 4250 50  0001 C CNN
+F 3 "~" H 9550 4250 50  0001 C CNN
+	1    9550 4250
+	1    0    0    -1
+$EndComp
+$Comp
+L power:+3V3 #PWR0187
+U 1 1 5EE14C63
+P 9550 4100
+F 0 "#PWR0187" H 9550 3950 50  0001 C CNN
+F 1 "+3V3" H 9400 4200 50  0000 C CNN
+F 2 "" H 9550 4100 50  0001 C CNN
+F 3 "" H 9550 4100 50  0001 C CNN
+	1    9550 4100
+	1    0    0    -1
+$EndComp
+$Comp
+L Device:R R?
+U 1 1 5EE24215
+P 9550 5200
+AR Path="/5EE24215" Ref="R?"  Part="1"
+AR Path="/5CFF3BEB/5EE24215" Ref="R94"  Part="1"
+F 0 "R94" H 9500 5250 50  0000 R CNN
+F 1 "10k" H 9500 5150 50  0000 R CNN
+F 2 "Resistor_BG:R_0805_2012Metric" V 9480 5200 50  0001 C CNN
+F 3 "~" H 9550 5200 50  0001 C CNN
+	1    9550 5200
+	1    0    0    -1
+$EndComp
+$Comp
+L power:+3V3 #PWR0188
+U 1 1 5EE2421B
+P 9550 5050
+F 0 "#PWR0188" H 9550 4900 50  0001 C CNN
+F 1 "+3V3" H 9565 5223 50  0000 C CNN
+F 2 "" H 9550 5050 50  0001 C CNN
+F 3 "" H 9550 5050 50  0001 C CNN
+	1    9550 5050
+	1    0    0    -1
+$EndComp
+$Comp
+L Device:R R?
+U 1 1 5EE331A1
+P 9550 5900
+AR Path="/5EE331A1" Ref="R?"  Part="1"
+AR Path="/5CFF3BEB/5EE331A1" Ref="R95"  Part="1"
+F 0 "R95" H 9500 5950 50  0000 R CNN
+F 1 "10k" H 9500 5850 50  0000 R CNN
+F 2 "Resistor_BG:R_0805_2012Metric" V 9480 5900 50  0001 C CNN
+F 3 "~" H 9550 5900 50  0001 C CNN
+	1    9550 5900
+	1    0    0    -1
+$EndComp
+$Comp
+L power:+3V3 #PWR0189
+U 1 1 5EE331A7
+P 9550 5750
+F 0 "#PWR0189" H 9550 5600 50  0001 C CNN
+F 1 "+3V3" H 9400 5850 50  0000 C CNN
+F 2 "" H 9550 5750 50  0001 C CNN
+F 3 "" H 9550 5750 50  0001 C CNN
+	1    9550 5750
+	1    0    0    -1
+$EndComp
+Connection ~ 9550 1500
 $EndSCHEMATC
