File: Hardware/Encoders&Buttons.sch (KiCad schematic (older format))
At the start: 132 parts, among them SW1 Rotary_Encoder_Switch, SW10 SW_Push_LED_Red, SW11 SW_Push_LED_Blue, SW12 SW_Push_LED_Red, SW13 SW_Push_LED_Yellow, SW14 SW_Push_LED_Green, SW15 SW_Push_LED_Blue, SW2 Rotary_Encoder_Switch, SW3 Rotary_Encoder_Switch, SW4 Rotary_Encoder_Switch, SW5 Rotary_Encoder_Switch, SW6 Rotary_Encoder_Switch, SW7 Rotary_Encoder_Switch, SW8 Rotary_Encoder_Switch, SW9 Rotary_Encoder_Switch, U18 74LVC14, U19 74LVC14, U20 74LVC14, U21 74LVC14, U22 74LVC14, U23 74LVC14

Commit message: Updated schematic and BOM spreadsheets with Manufacturer and Part Numbers
Parts:
- C12, C13, C16, C17, C21, C22, C23, C24, C29, C42, C43, C44, C48, C49, C50, C51, C55, C56: MFR (none) -> Samsung; MPN (none) -> CL21B103KCANNNC
- C14, C15, C18, C19, C20, C25, C26, C27, C28, C45, C46, C47, C52, C53, C54, C57, C58, C59, C60, C61, C62: MFR (none) -> Samsung; MPN (none) -> CL21B104KBCNFNC
- R22, R23, R24, R25, R27, R28, R29, R30, R32, R33, R34, R35, R36, R37, R39, R40, R42, R43, R44, R45, R46, R47, R49, R50, R52, R53, R54, R55, R56, R57, R58, R59, R60, R61, R62, R63, R64, R65, R66, R67, R68, R69, R70, R71, R72, R73, R74, R75, R76, R77, R78, R79, R80, R81, R82, R83, R84, R85, R86, R87, R90, R91, R92, R93, R94, R95: MFR (none) -> Yageo; MPN (none) -> RC0805FR-0710KL
- R26, R38: MFR (none) -> Yageo; MPN (none) -> RC0805FR-07150RL
- R31, R51: MFR (none) -> Yageo; MPN (none) -> RC0805FR-0733RL
- R41, R48: MFR (none) -> Yageo; MPN (none) -> RC0805FR-07120RL
- SW1, SW2, SW3, SW4, SW5, SW6, SW7, SW8, SW9: MFR (none) -> Bourns Inc.; MPN (none) -> PEC12R-4025F-S0024
- SW10: MFR (none) -> E-Switch; MPN (none) -> TL3240F160R;TL3240R1CAPBLK
- SW11: MFR (none) -> E-Switch; MPN (none) -> TL3240F160B;TL3240R1CAPBLU
- SW12: MFR (none) -> E-Switch; MPN (none) -> TL3240F160R;TL3240S1CAPIVR
- SW13: MFR (none) -> E-Switch; MPN (none) -> TL3240F160Y;TL3240S1CAPIVR
- SW14: MFR (none) -> E-Switch; MPN (none) -> TL3240F160G;TL3240S1CAPIVR
- SW15: MFR (none) -> E-Switch; MPN (none) -> TL3240F160B;TL3240S1CAPIVR
- U18, U19, U20, U21, U22, U23: MFR (none) -> Texas Instruments; MPN (none) -> SN74LVC14ADR
