File: Hardware/Encoders&Buttons.sch (KiCad schematic (older format))
At the start: 132 parts, among them SW1 Rotary_Encoder_Switch, SW10 SW_Push_LED_Red, SW11 SW_Push_LED_Blue, SW12 SW_Push_LED_Red, SW13 SW_Push_LED_Yellow, SW14 SW_Push_LED_Green, SW15 SW_Push_LED_Blue, SW2 Rotary_Encoder_Switch, SW3 Rotary_Encoder_Switch, SW4 Rotary_Encoder_Switch, SW5 Rotary_Encoder_Switch, SW6 Rotary_Encoder_Switch, SW7 Rotary_Encoder_Switch, SW8 Rotary_Encoder_Switch, SW9 Rotary_Encoder_Switch, U18 74LVC14, U19 74LVC14, U20 74LVC14, U21 74LVC14, U22 74LVC14, U23 74LVC14

Commit message: Applied MPN to each item and consolidated some parts
Parts:
- C12, C13, C16, C17, C21, C22, C23, C24, C29, C42, C43, C44, C48, C49, C50, C51, C55, C56: value 10nF -> 0.01uF; MFR (none) -> Samsung; MPN (none) -> CL21B103KCANNNC; Seeed OPL (none) -> CC0805JRX7R9BB103; Seeed OPL SKU (none) -> 302010175
- C14, C15, C18, C19, C20, C25, C26, C27, C28, C45, C46, C47, C52, C53, C54, C57, C58, C59, C60, C61, C62: value 100nF -> 0.1uF; MFR (none) -> Samsung; MPN (none) -> CL21B104KBCNFNC; Seeed OPL (none) -> CC0805KRX7R9BB104; Seeed OPL SKU (none) -> 302010165
- R22, R23, R24, R25, R27, R28, R29, R30, R32, R33, R34, R35, R36, R37, R39, R40, R42, R43, R44, R45, R46, R47, R49, R50, R52, R53, R54, R55, R56, R57, R58, R59, R60, R61, R62, R63, R64, R65, R66, R67, R68, R69, R70, R71, R72, R73, R74, R75, R76, R77, R78, R79, R80, R81, R82, R83, R84, R85, R86, R87, R90, R91, R92, R93, R94, R95: MFR (none) -> Yageo; MPN (none) -> RC0805FR-0710KL; Seeed OPL (none) -> RC0805FR-0710KL; Seeed OPL SKU (none) -> 301010361
- R26, R38: value 150 -> 150R; MFR (none) -> Yageo; MPN (none) -> RC0805FR-07150RL; Seeed OPL (none) -> RC0805FR-07150RL; Seeed OPL SKU (none) -> 301010370
- R31, R51: value 33 -> 33R; MFR (none) -> Yageo; MPN (none) -> RC0805FR-0733RL; Seeed OPL (none) -> RC0805FR-0733RL; Seeed OPL SKU (none) -> 301012298
- R41, R48: value 120 -> 150R; MFR (none) -> Yageo; MPN (none) -> RC0805FR-07150RL; Seeed OPL (none) -> RC0805FR-07150RL; Seeed OPL SKU (none) -> 301010370
- SW1, SW2, SW3, SW4, SW5, SW6, SW7, SW8, SW9: value Rotary_Encoder_Switch -> Encoder_SW_D12.0xH25.0mm; DNP (none) -> DNP; MFR (none) -> Bourns; MPN (none) -> PEC12R-4025F-S0024-ND
- SW10: DNP (none) -> DNP; MFR (none) -> E-Switch; MPN (none) -> TL3240F160R;TL3240R1CAPBLK
- SW11: DNP (none) -> DNP; MFR (none) -> E-Switch; MPN (none) -> TL3240F160B;TL3240R1CAPBLU
- SW12: DNP (none) -> DNP; MFR (none) -> E-Switch; MPN (none) -> TL3240F160R;TL3240S1CAPIVR
- SW13: DNP (none) -> DNP; MFR (none) -> E-Switch; MPN (none) -> TL3240F160Y;TL3240S1CAPIVR
- SW14: DNP (none) -> DNP; MFR (none) -> E-Switch; MPN (none) -> TL3240F160G;TL3240S1CAPIVR
- SW15: DNP (none) -> DNP; MFR (none) -> E-Switch; MPN (none) -> TL3240F160B;TL3240S1CAPIVR
- U18, U19, U20, U21, U22, U23: MFR (none) -> Texas Instruments; MPN (none) -> SN74LVC14ADR; Seeed OPL (none) -> 74LVC14AD,118; Seeed OPL SKU (none) -> 74LVC14AD,118

Commit message: Substituted buttons as digikey is discontinuing the old ones.
Still need to update their footprints.
Parts:
- SW10: footprint Button_Switch_BG:E-Switch_SPST_Red_LED_RoundCap_TL3240F160R -> (none); MFR E-Switch -> TE Connectivity; MPN TL3240F160R;TL3240R1CAPBLK -> FSMIJ63BR04;2311402-2
- SW11: footprint Button_Switch_BG:E-Switch_SPST_LED_RoundCap_TL3240F160x -> (none); MFR E-Switch -> TE Connectivity; MPN TL3240F160B;TL3240R1CAPBLU -> FSMIJ63BB04;2311402-4
- SW12: footprint Button_Switch_BG:E-Switch_SPST_Red_LED_SquareCap_TL3240F160R -> (none); MFR E-Switch -> TE Connectivity; MPN TL3240F160R;TL3240S1CAPIVR -> FSMIJ63BR04;2311403-2
- SW13: footprint Button_Switch_BG:E-Switch_SPST_LED_SquareCap_TL3240F160x -> (none); MFR E-Switch -> TE Connectivity; MPN TL3240F160Y;TL3240S1CAPIVR -> FSMIJ63BA04;2311403-2
- SW14: footprint Button_Switch_BG:E-Switch_SPST_LED_SquareCap_TL3240F160x -> (none); MFR E-Switch -> TE Connectivity; MPN TL3240F160G;TL3240S1CAPIVR -> FSMIJ63BG04;2311403-2
- SW15: footprint Button_Switch_BG:E-Switch_SPST_LED_SquareCap_TL3240F160x -> (none); MFR E-Switch -> TE Connectivity; MPN TL3240F160B;TL3240S1CAPIVR -> FSMIJ63BB04;2311403-2
Changed lines of the file:
@@
 F 0 "SW12" H 8850 4185 50  0000 C CNN
 F 1 "SW_Push_LED_Red" H 8850 4094 50  0000 C CNN
-F 2 "Button_Switch_BG:E-Switch_SPST_Red_LED_SquareCap_TL3240F160R" H 8850 4100 50  0001 C CNN
-F 3 "https://sten-eswitch-13110800-production.s3.amazonaws.com/system/asset/product_line/data_sheet/155/TL3240.pdf" H 8850 4100 50  0001 C CNN
-F 4 "E-Switch" H 8850 3800 50  0001 C CNN "MFR"
-F 5 "TL3240F160R;TL3240S1CAPIVR" H 8850 3800 50  0001 C CNN "MPN"
+F 2 "" H 8850 4100 50  0001 C CNN
+F 3 "https://www.te.com/commerce/DocumentDelivery/DDEController?Action=srchrtrv&DocNm=1-1773878-5_IlluminatedTactileSwitch&DocType=DS&DocLang=English" H 8850 4100 50  0001 C CNN
+F 4 "TE Connectivity" H 8850 3800 50  0001 C CNN "MFR"
+F 5 "FSMIJ63BR04;2311403-2" H 8850 3800 50  0001 C CNN "MPN"
 F 6 "DNP" H 8850 3800 50  0001 C CNN "DNP"
 	1    8850 3800
@@
 F 0 "SW13" H 8850 4885 50  0000 C CNN
 F 1 "SW_Push_LED_Yellow" H 8850 4794 50  0000 C CNN
-F 2 "Button_Switch_BG:E-Switch_SPST_LED_SquareCap_TL3240F160x" H 8850 4800 50  0001 C CNN
-F 3 "https://sten-eswitch-13110800-production.s3.amazonaws.com/system/asset/product_line/data_sheet/155/TL3240.pdf" H 8850 4800 50  0001 C CNN
-F 4 "E-Switch" H 8850 4500 50  0001 C CNN "MFR"
-F 5 "TL3240F160Y;TL3240S1CAPIVR" H 8850 4500 50  0001 C CNN "MPN"
+F 2 "" H 8850 4800 50  0001 C CNN
+F 3 "https://www.te.com/commerce/DocumentDelivery/DDEController?Action=srchrtrv&DocNm=1-1773878-5_IlluminatedTactileSwitch&DocType=DS&DocLang=English" H 8850 4800 50  0001 C CNN
+F 4 "TE Connectivity" H 8850 4500 50  0001 C CNN "MFR"
+F 5 "FSMIJ63BA04;2311403-2" H 8850 4500 50  0001 C CNN "MPN"
 F 6 "DNP" H 8850 4500 50  0001 C CNN "DNP"
 	1    8850 4500
@@
 F 0 "SW14" H 8850 5835 50  0000 C CNN
 F 1 "SW_Push_LED_Green" H 8850 5744 50  0000 C CNN
-F 2 "Button_Switch_BG:E-Switch_SPST_LED_SquareCap_TL3240F160x" H 8850 5750 50  0001 C CNN
-F 3 "https://sten-eswitch-13110800-production.s3.amazonaws.com/system/asset/product_line/data_sheet/155/TL3240.pdf" H 8850 5750 50  0001 C CNN
-F 4 "E-Switch" H 8850 5450 50  0001 C CNN "MFR"
-F 5 "TL3240F160G;TL3240S1CAPIVR" H 8850 5450 50  0001 C CNN "MPN"
+F 2 "" H 8850 5750 50  0001 C CNN
+F 3 "https://www.te.com/commerce/DocumentDelivery/DDEController?Action=srchrtrv&DocNm=1-1773878-5_IlluminatedTactileSwitch&DocType=DS&DocLang=English" H 8850 5750 50  0001 C CNN
+F 4 "TE Connectivity" H 8850 5450 50  0001 C CNN "MFR"
+F 5 "FSMIJ63BG04;2311403-2" H 8850 5450 50  0001 C CNN "MPN"
 F 6 "DNP" H 8850 5450 50  0001 C CNN "DNP"
 	1    8850 5450
@@
 F 0 "SW15" H 8850 6535 50  0000 C CNN
 F 1 "SW_Push_LED_Blue" H 8850 6444 50  0000 C CNN
-F 2 "Button_Switch_BG:E-Switch_SPST_LED_SquareCap_TL3240F160x" H 8850 6450 50  0001 C CNN
-F 3 "https://sten-eswitch-13110800-production.s3.amazonaws.com/system/asset/product_line/data_sheet/155/TL3240.pdf" H 8850 6450 50  0001 C CNN
-F 4 "E-Switch" H 8850 6150 50  0001 C CNN "MFR"
-F 5 "TL3240F160B;TL3240S1CAPIVR" H 8850 6150 50  0001 C CNN "MPN"
+F 2 "" H 8850 6450 50  0001 C CNN
+F 3 "https://www.te.com/commerce/DocumentDelivery/DDEController?Action=srchrtrv&DocNm=1-1773878-5_IlluminatedTactileSwitch&DocType=DS&DocLang=English" H 8850 6450 50  0001 C CNN
+F 4 "TE Connectivity" H 8850 6150 50  0001 C CNN "MFR"
+F 5 "FSMIJ63BB04;2311403-2" H 8850 6150 50  0001 C CNN "MPN"
 F 6 "DNP" H 8850 6150 50  0001 C CNN "DNP"
 	1    8850 6150
@@
 F 0 "SW11" H 8850 3235 50  0000 C CNN
 F 1 "SW_Push_LED_Blue" H 8850 3144 50  0000 C CNN
-F 2 "Button_Switch_BG:E-Switch_SPST_LED_RoundCap_TL3240F160x" H 8850 3150 50  0001 C CNN
-F 3 "https://sten-eswitch-13110800-production.s3.amazonaws.com/system/asset/product_line/data_sheet/155/TL3240.pdf" H 8850 3150 50  0001 C CNN
-F 4 "E-Switch" H 8850 2850 50  0001 C CNN "MFR"
-F 5 "TL3240F160B;TL3240R1CAPBLU" H 8850 2850 50  0001 C CNN "MPN"
+F 2 "" H 8850 3150 50  0001 C CNN
+F 3 "https://www.te.com/commerce/DocumentDelivery/DDEController?Action=srchrtrv&DocNm=1-1773878-5_IlluminatedTactileSwitch&DocType=DS&DocLang=English" H 8850 3150 50  0001 C CNN
+F 4 "TE Connectivity" H 8850 2850 50  0001 C CNN "MFR"
+F 5 "FSMIJ63BB04;2311402-4" H 8850 2850 50  0001 C CNN "MPN"
 F 6 "DNP" H 8850 2850 50  0001 C CNN "DNP"
 	1    8850 2850
@@
 F 0 "SW10" H 8850 1985 50  0000 C CNN
 F 1 "SW_Push_LED_Red" H 8850 1894 50  0000 C CNN
-F 2 "Button_Switch_BG:E-Switch_SPST_Red_LED_RoundCap_TL3240F160R" H 8850 1900 50  0001 C CNN
-F 3 "https://sten-eswitch-13110800-production.s3.amazonaws.com/system/asset/product_line/data_sheet/155/TL3240.pdf" H 8850 1900 50  0001 C CNN
-F 4 "E-Switch" H 8850 1600 50  0001 C CNN "MFR"
-F 5 "TL3240F160R;TL3240R1CAPBLK" H 8850 1600 50  0001 C CNN "MPN"
+F 2 "" H 8850 1900 50  0001 C CNN
+F 3 "https://www.te.com/commerce/DocumentDelivery/DDEController?Action=srchrtrv&DocNm=1-1773878-5_IlluminatedTactileSwitch&DocType=DS&DocLang=English" H 8850 1900 50  0001 C CNN
+F 4 "TE Connectivity" H 8850 1600 50  0001 C CNN "MFR"
+F 5 "FSMIJ63BR04;2311402-2" H 8850 1600 50  0001 C CNN "MPN"
 F 6 "DNP" H 8850 1600 50  0001 C CNN "DNP"
 	1    8850 1600

Commit message: Finished (untested) sketch of the Rev C PCB.
TODO: Revise svg, 3D model and PDFs of the acrylic.
Parts:
- R31, R51: value 33R -> 150R; MPN RC0805FR-0733RL -> RC0805FR-07150RL; Seeed OPL RC0805FR-0733RL -> RC0805FR-07150RL; Seeed OPL SKU 301012298 -> 301010370
- SW10, SW11, SW12, SW13, SW14, SW15: footprint (none) -> Button_Switch_BG:TE_Alcoswitch_SPST_LED
Connections:
- net GND: now also SW10.2, SW11.2, SW12.2, SW13.2, SW14.2, SW15.2
- net at R53.2, R91.2, SW11.3: now also SW11.4
- net at R36.2, R90.2, SW10.3: now also SW10.4
- net at R64.2, R92.2, SW12.3: now also SW12.4
- net at R67.2, R93.2, SW13.3: now also SW13.4
- net at R80.2, R94.2, SW14.3: now also SW14.4
- net at R86.2, R95.2, SW15.3: now also SW15.4
- no-connect marks 12 -> 0
Changed lines of the file:
@@
 Sheet 2 3
 Title "Encoder Board"
-Date "2020-06-03"
-Rev "C-dev"
+Date "2020-06-10"
+Rev "C"
 Comp "Blake Garner"
 Comment1 ""
@@
 F 0 "SW12" H 8850 4185 50  0000 C CNN
 F 1 "SW_Push_LED_Red" H 8850 4094 50  0000 C CNN
-F 2 "" H 8850 4100 50  0001 C CNN
+F 2 "Button_Switch_BG:TE_Alcoswitch_SPST_LED" H 8850 4100 50  0001 C CNN
 F 3 "https://www.te.com/commerce/DocumentDelivery/DDEController?Action=srchrtrv&DocNm=1-1773878-5_IlluminatedTactileSwitch&DocType=DS&DocLang=English" H 8850 4100 50  0001 C CNN
 F 4 "TE Connectivity" H 8850 3800 50  0001 C CNN "MFR"
@@
 F 0 "SW13" H 8850 4885 50  0000 C CNN
 F 1 "SW_Push_LED_Yellow" H 8850 4794 50  0000 C CNN
-F 2 "" H 8850 4800 50  0001 C CNN
+F 2 "Button_Switch_BG:TE_Alcoswitch_SPST_LED" H 8850 4800 50  0001 C CNN
 F 3 "https://www.te.com/commerce/DocumentDelivery/DDEController?Action=srchrtrv&DocNm=1-1773878-5_IlluminatedTactileSwitch&DocType=DS&DocLang=English" H 8850 4800 50  0001 C CNN
 F 4 "TE Connectivity" H 8850 4500 50  0001 C CNN "MFR"
@@
 F 0 "SW14" H 8850 5835 50  0000 C CNN
 F 1 "SW_Push_LED_Green" H 8850 5744 50  0000 C CNN
-F 2 "" H 8850 5750 50  0001 C CNN
+F 2 "Button_Switch_BG:TE_Alcoswitch_SPST_LED" H 8850 5750 50  0001 C CNN
 F 3 "https://www.te.com/commerce/DocumentDelivery/DDEController?Action=srchrtrv&DocNm=1-1773878-5_IlluminatedTactileSwitch&DocType=DS&DocLang=English" H 8850 5750 50  0001 C CNN
 F 4 "TE Connectivity" H 8850 5450 50  0001 C CNN "MFR"
@@
 F 0 "SW15" H 8850 6535 50  0000 C CNN
 F 1 "SW_Push_LED_Blue" H 8850 6444 50  0000 C CNN
-F 2 "" H 8850 6450 50  0001 C CNN
+F 2 "Button_Switch_BG:TE_Alcoswitch_SPST_LED" H 8850 6450 50  0001 C CNN
 F 3 "https://www.te.com/commerce/DocumentDelivery/DDEController?Action=srchrtrv&DocNm=1-1773878-5_IlluminatedTactileSwitch&DocType=DS&DocLang=English" H 8850 6450 50  0001 C CNN
 F 4 "TE Connectivity" H 8850 6150 50  0001 C CNN "MFR"
@@
 P 8350 6250
 F 0 "R51" V 8143 6250 50  0000 C CNN
-F 1 "33R" V 8234 6250 50  0000 C CNN
+F 1 "150R" V 8234 6250 50  0000 C CNN
 F 2 "Resistor_BG:R_0805_2012Metric" V 8280 6250 50  0001 C CNN
 F 3 "https://www.yageo.com/upload/media/product/productsearch/datasheet/rchip/PYu-RC_Group_51_RoHS_L_10.pdf" H 8350 6250 50  0001 C CNN
 F 4 "Yageo" H 8350 6250 50  0001 C CNN "MFR"
-F 5 "RC0805FR-0733RL" H 8350 6250 50  0001 C CNN "MPN"
-F 6 "RC0805FR-0733RL" H 8350 6250 50  0001 C CNN "Seeed OPL"
-F 7 "301012298" H 8350 6250 50  0001 C CNN "Seeed OPL SKU"
+F 5 "RC0805FR-07150RL" H 8350 6250 50  0001 C CNN "MPN"
+F 6 "RC0805FR-07150RL" H 8350 6250 50  0001 C CNN "Seeed OPL"
+F 7 "301010370" H 8350 6250 50  0001 C CNN "Seeed OPL SKU"
 	1    8350 6250
 	0    1    1    0
@@
 F 0 "SW11" H 8850 3235 50  0000 C CNN
 F 1 "SW_Push_LED_Blue" H 8850 3144 50  0000 C CNN
-F 2 "" H 8850 3150 50  0001 C CNN
+F 2 "Button_Switch_BG:TE_Alcoswitch_SPST_LED" H 8850 3150 50  0001 C CNN
 F 3 "https://www.te.com/commerce/DocumentDelivery/DDEController?Action=srchrtrv&DocNm=1-1773878-5_IlluminatedTactileSwitch&DocType=DS&DocLang=English" H 8850 3150 50  0001 C CNN
 F 4 "TE Connectivity" H 8850 2850 50  0001 C CNN "MFR"
@@
 F 0 "SW10" H 8850 1985 50  0000 C CNN
 F 1 "SW_Push_LED_Red" H 8850 1894 50  0000 C CNN
-F 2 "" H 8850 1900 50  0001 C CNN
+F 2 "Button_Switch_BG:TE_Alcoswitch_SPST_LED" H 8850 1900 50  0001 C CNN
 F 3 "https://www.te.com/commerce/DocumentDelivery/DDEController?Action=srchrtrv&DocNm=1-1773878-5_IlluminatedTactileSwitch&DocType=DS&DocLang=English" H 8850 1900 50  0001 C CNN
 F 4 "TE Connectivity" H 8850 1600 50  0001 C CNN "MFR"
@@
 P 8350 2950
 F 0 "R31" V 8143 2950 50  0000 C CNN
-F 1 "33R" V 8234 2950 50  0000 C CNN
+F 1 "150R" V 8234 2950 50  0000 C CNN
 F 2 "Resistor_BG:R_0805_2012Metric" V 8280 2950 50  0001 C CNN
 F 3 "https://www.yageo.com/upload/media/product/productsearch/datasheet/rchip/PYu-RC_Group_51_RoHS_L_10.pdf" H 8350 2950 50  0001 C CNN
 F 4 "Yageo" H 8350 2950 50  0001 C CNN "MFR"
-F 5 "RC0805FR-0733RL" H 8350 2950 50  0001 C CNN "MPN"
-F 6 "RC0805FR-0733RL" H 8350 2950 50  0001 C CNN "Seeed OPL"
-F 7 "301012298" H 8350 2950 50  0001 C CNN "Seeed OPL SKU"
+F 5 "RC0805FR-07150RL" H 8350 2950 50  0001 C CNN "MPN"
+F 6 "RC0805FR-07150RL" H 8350 2950 50  0001 C CNN "Seeed OPL"
+F 7 "301010370" H 8350 2950 50  0001 C CNN "Seeed OPL SKU"
 	1    8350 2950
 	0    1    1    0
@@
 Wire Wire Line
 	8050 6050 8650 6050
-NoConn ~ 9050 6150
-NoConn ~ 8650 6150
-NoConn ~ 8650 5450
-NoConn ~ 9050 5450
-NoConn ~ 9050 4500
-NoConn ~ 8650 4500
-NoConn ~ 8650 3800
-NoConn ~ 9050 3800
-NoConn ~ 9050 2850
-NoConn ~ 8650 2850
-NoConn ~ 8650 1600
-NoConn ~ 9050 1600
 $Comp
 L Device:R R?
@@
 $EndComp
 Connection ~ 9550 1500
+Wire Wire Line
+	9050 1600 9050 1500
+Connection ~ 9050 1500
+Wire Wire Line
+	8650 1600 8650 1500
+Connection ~ 8650 1500
+Wire Wire Line
+	9050 6150 9050 6050
+Connection ~ 9050 6050
+Wire Wire Line
+	8650 6150 8650 6050
+Connection ~ 8650 6050
+Wire Wire Line
+	8650 5450 8650 5350
+Connection ~ 8650 5350
+Wire Wire Line
+	9050 5450 9050 5350
+Connection ~ 9050 5350
+Wire Wire Line
+	8650 4500 8650 4400
+Connection ~ 8650 4400
+Wire Wire Line
+	9050 4500 9050 4400
+Connection ~ 9050 4400
+Wire Wire Line
+	9050 3800 9050 3700
+Connection ~ 9050 3700
+Wire Wire Line
+	8650 3800 8650 3700
+Connection ~ 8650 3700
+Wire Wire Line
+	8650 2850 8650 2750
+Connection ~ 8650 2750
+Wire Wire Line
+	9050 2850 9050 2750
+Connection ~ 9050 2750
 $EndSCHEMATC
