File: Hardware/Displays&LEDs.sch (KiCad schematic (older format))
At the start: 42 parts, among them U10 Display_OLED_128x32_I2C, U11 Display_OLED_128x32_I2C, U12 Display_OLED_128x32_I2C, U13 Display_OLED_128x32_I2C, U14 Display_OLED_128x32_I2C, U15 Display_OLED_128x32_I2C, U16 Display_OLED_128x32_I2C, U17 Display_OLED_128x32_I2C, U9 Display_OLED_128x32_I2C

Commit message: Updated schematic and BOM spreadsheets with Manufacturer and Part Numbers
Parts:
- C30, C31, C32, C33, C34, C35, C36, C37, C38, C39, C40, C41, C63, C64, C65, C66, C67, C68, C69, C70, C71: MFR (none) -> Samsung; MPN (none) -> CL21B104KBCNFNC
- D1, D10, D11, D12, D2, D3, D4, D5, D6, D7, D8, D9: MFR (none) -> World Semi; MPN (none) -> WS2812B
- U10, U11, U12, U13, U14, U15, U16, U17, U9: MFR (none) -> Unbranded; MPN (none) -> 128x32_I2C_OLED_SSD1306
