File: Hardware/Displays&LEDs.sch (KiCad schematic (older format))
At the start: 42 parts, among them U10 Display_OLED_128x32_I2C, U11 Display_OLED_128x32_I2C, U12 Display_OLED_128x32_I2C, U13 Display_OLED_128x32_I2C, U14 Display_OLED_128x32_I2C, U15 Display_OLED_128x32_I2C, U16 Display_OLED_128x32_I2C, U17 Display_OLED_128x32_I2C, U9 Display_OLED_128x32_I2C

Commit message: Applied MPN to each item and consolidated some parts
Parts:
- C30, C31, C32, C33, C34, C35, C36, C37, C38, C39, C40, C41, C63, C64, C65, C66, C67, C68, C69, C70, C71: value 100nF -> 0.1uF; MFR (none) -> Samsung; MPN (none) -> CL21B104KBCNFNC; Seeed OPL (none) -> CC0805KRX7R9BB104; Seeed OPL SKU (none) -> 302010165
- D1, D10, D11, D12, D2, D3, D4, D5, D6, D7, D8, D9: MFR (none) -> WorldSemi; MPN (none) -> WS2812B; Seeed OPL (none) -> WS2812B; Seeed OPL SKU (none) -> 304990003
- U10, U11, U12, U13, U14, U15, U16, U17, U9: DNP (none) -> DNP; MFR (none) -> Unbranded; MPN (none) -> SSD1306_I2C_128x32_OLED
