File: Hardware/EncoderBoard.sch (KiCad schematic (older format))
At the start: 49 parts, among them U1 MCP23S17_SO, U2 MCP23S17_SO, U24 CAT24M01W, U25 CAT24M01W, U26 CAT24M01W, U3 MCP23S17_SO, U4 TCA9548APWR, U5 74HCT245, U6 TCA9548APWR, U7 Teensy3.2, U8 CAT24M01W

Commit message: Applied MPN to each item and consolidated some parts
Parts:
- added R96: 150R, Resistor_BG:R_0805_2012Metric, symbol Device:R
- C1, C10, C3, C5, C7, C72, C73, C74, C75, C9: value 100nF -> 0.1uF; MFR (none) -> Samsung; MPN (none) -> CL21B104KBCNFNC; Seeed OPL (none) -> CC0805KRX7R9BB104; Seeed OPL SKU (none) -> 302010165
- C11, C2, C4, C6, C8: MFR (none) -> Samsung; MPN (none) -> CL32B106KOJNNNE; Seeed OPL (none) -> CC1206KKX5R8BB106; Seeed OPL SKU (none) -> 302010181
- R1, R10, R11, R12, R13, R14, R15, R16, R18, R19, R2, R20, R21, R3, R4, R5, R6, R7, R8, R88, R89, R9: MFR (none) -> Yageo; MPN (none) -> RC0805FR-074K7L; Seeed OPL (none) -> RC0805FR-074K7L; Seeed OPL SKU (none) -> 301010336
- R17: value 330R -> 150R; MFR (none) -> Yageo; MPN (none) -> RC0805FR-07150RL; Seeed OPL (none) -> RC0805FR-07150RL; Seeed OPL SKU (none) -> 301010370
- U1, U2, U3: MFR (none) -> Microchip; MPN (none) -> MCP23S17T-E/SO
- U24, U25, U26, U8: MFR (none) -> ON Semiconductor; MPN (none) -> CAT24M01WI-GT3
- U4, U6: symbol Interface_Expansion:TCA9548APWR -> EncoderBoard-rescue:TCA9548APWR-Interface_Expansion; MFR (none) -> Texas Instruments; MPN (none) -> TCA9548APWR
- U5: MFR (none) -> Texas Instruments; MPN (none) -> SN74HCT245DWR; Seeed OPL (none) -> 74HCT245D,653; Seeed OPL SKU (none) -> 74HCT245D,653
- U7: DNP (none) -> DNP; MFR (none) -> PJRC; MPN (none) -> TEENSY32
Connections:
- net WS2812_DATA: now also R96.1; no longer R17.1
- new net: R17.1, R96.2

Commit message: Substituted buttons as digikey is discontinuing the old ones.
Still need to update their footprints.
Changed lines of the file:
@@
 F 1 "Teensy3.2" H 2700 7581 60  0000 C CNN
 F 2 "Teensy_BG:Teensy30_31_32_LC" H 2700 5300 60  0001 C CNN
-F 3 "https://www.pjrc.com/store/teensy32.html" H 2700 5300 60  0000 C CNN
+F 3 "https://www.pjrc.com/store/teensy32.html" H 2700 5300 60  0001 C CNN
 F 4 "PJRC" H 2700 6100 50  0001 C CNN "MFR"
 F 5 "TEENSY32" H 2700 6100 50  0001 C CNN "MPN"
