File: Hardware/EncoderBoard.sch (KiCad schematic (older format))
At the start: 49 parts, among them U1 MCP23S17_SO, U2 MCP23S17_SO, U24 CAT24M01W, U25 CAT24M01W, U26 CAT24M01W, U3 MCP23S17_SO, U4 TCA9548APWR, U5 74HCT245, U6 TCA9548APWR, U7 Teensy3.2, U8 CAT24M01W

Commit message: Updated schematic and BOM spreadsheets with Manufacturer and Part Numbers
Parts:
- C1, C10, C3, C5, C7, C72, C73, C74, C75, C9: MFR (none) -> Samsung; MPN (none) -> CL21B104KBCNFNC
- C11, C2, C4, C6, C8: MFR (none) -> Samsung; MPN (none) -> CL32B106KPINNNE
- R1, R10, R11, R12, R13, R14, R15, R16, R18, R19, R2, R20, R21, R3, R4, R5, R6, R7, R8, R88, R89, R9: MFR (none) -> Yageo; MPN (none) -> RC0805FR-074K7L
- R17: MFR (none) -> Yageo; MPN (none) -> RC0805FR-07330RL
- U1, U2, U3: MFR (none) -> Microchip; MPN (none) -> MCP23S17T-E/SO
- U24, U25, U26, U8: MFR (none) -> ON Semiconductor; MPN (none) -> CAT24M01WI-GT3
- U4, U6: MFR (none) -> Texas Instruments; MPN (none) -> TCA9548APWR
- U5: MFR (none) -> Texas Instruments; MPN (none) -> SN74HCT245DWR
- U7: MFR (none) -> PJRC; MPN (none) -> TEENSY32

Commit message: Fixed incorrect package in SN74HCT245. Should have been TSSOP instead of SOIP.
Parts:
- U5: MPN SN74HCT245DWR -> SN74HCT245PWR
Changed lines of the file:
@@
 F 3 "http://www.ti.com/lit/gpn/sn74HC245" H 5100 4500 50  0001 C CNN
 F 4 "Texas Instruments" H 5100 4500 50  0001 C CNN "MFR"
-F 5 "SN74HCT245DWR" H 5100 4500 50  0001 C CNN "MPN"
+F 5 "SN74HCT245PWR" H 5100 4500 50  0001 C CNN "MPN"
 	1    5100 4500
 	1    0    0    -1
